File: mls800.sch (KiCad schematic (older format))
At the start: 37 parts

Commit message: MLS800  * Lots of change in diagram/schematic  * Added external parts
Parts:
- removed CN?: CN_USB, adafruit-USB-MINIB, symbol CN_USB
- removed D?: blue, ~, symbol LED
- removed D?: green, ~, symbol LED
- removed R? (x2): 10K, ~, symbol R
- removed R? (x2): 1K, ~, symbol R
- removed S? (x2): SW_TACT, ~, symbol SW_TACT
- removed SHIELD?: ARDUINO_SHIELD, ~, symbol ARDUINO_SHIELD
- added C2: 1uF, ~, symbol C
- added D5: DIODE, ~, symbol DIODE
- added FB1: FILTER, ~, symbol FILTER
- added IC1: 6N137, DIP8, symbol 6N137
- added P1, P2: DIN_5, symbol DIN_5
- added R10, R8: 1K, ~, symbol R
- added R11, R9: 10K, ~, symbol R
- added R12, R13, R14: 220R, ~, symbol R
- added S1, S2: SW_TACT_LED, ~, symbol SW_TACT_LED
- added U3: 24LC256, symbol 24LC256
- added X1: USBMICRO, symbol USBMICRO
- U1: renamed from U?; value 7805 -> LM340-5.0
- gave numbers to parts that had none: 26
Connections:
- net labels added: EDIT, EXIT
- wire segments 73 -> 107
Other:
- note added: "MEM\n"
- note added: "MIDI\n"
- note removed: "Add a filter if ADC is used ! (datasheet p7)"
- moved on the sheet: C1, C10, C8, C9, CON1, D2, D3, D4, F1, R2, R3, R4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

Commit message: MLS800  * Fixed missing non connected symbols
Parts:
- renumbered X1 to X2
Connections:
- wire segments 107 -> 111
- no-connect marks 0 -> 23

Commit message: MLS800  * Fixed some crc errors  * Fixed wrong AREF/UCAP schematics  * Generated netlist
Parts:
- added C8: 100nF, ~, symbol C
- renumbered C3 to C1, C9 to C10, C10 to C11, C4 to C2, C1 to C3, C2 to C4, C8 to C9
Connections:
- no-connect marks 23 -> 22
Other:
- note added: "Vérifier les condos. OK pour 7805 mais lm340 semble utilisé des céramiques de 0.1uF"
- moved on the sheet: C1, C2, X1

Commit message: MLS800  * Added separated GND : AGND & GND  * Revamped the loops schema  * Put values on all components  * Started to add footprint annotations to some resistors
Parts:
- removed C3, C9: CAPAPOL, ~, symbol CAPAPOL
- removed S1, S2: SW_TACT_LED, ~, symbol SW_TACT_LED
- added C3: 0.22uF, ~, symbol C
- added C9: 0.1uF, ~, symbol C
- added R25, R26: 0, ~, symbol R
- added SW18, SW19: SW_TACT_LED_2, symbol SW_TACT_LED_2
- D1, D5: value DIODE -> 1N4148
- D2: value DIODE -> 1N4001
- D3: value yellow -> Yellow
- D4: value yellow -> Red
- FB1: value FILTER -> MH2029-300Y
- R1, R4: value 10K -> 10k
- R10, R5, R6, R8: value 1K -> 1k; footprint ~ -> SM0805
- R11, R7, R9: value 10K -> 10k; footprint ~ -> SM0805
- X1: value CRYSTAL -> 16Mhz
Connections:
- net labels added: AGND, DGND, RXLED, TXLED
- wire segments 111 -> 116
Other:
- note removed: "Vérifier les condos. OK pour 7805 mais lm340 semble utilisé des céramiques de 0.1uF"

Commit message: MLS800  * Started cmp association
Parts:
- R10: renamed from R8; footprint SM0805 -> ~
- R11: renamed from R9; footprint SM0805 -> ~
- R12: renamed from R10; footprint SM0805 -> ~
- R13: renamed from R11; footprint SM0805 -> ~
- R7: renamed from R5; footprint SM0805 -> ~
- R8: renamed from R6; footprint SM0805 -> ~
- R9: renamed from R7; footprint SM0805 -> ~
- renumbered R12 to R14, R13 to R15, R14 to R16, R25 to R2, R26 to R3, R2 to R4, R3 to R5, R4 to R6, SW18 to SW2, SW19 to SW3

Commit message: MLS800 :  - assigning footprints
Parts:
- removed J1: 3X2M, symbol 3X2M
- added P3: CONN_02X03, Pin_Headers:Pin_Header_Straight_2x03, symbol CONN_02X03
- C1, C11, C3, C4, C5, C6, C7, C8, C9: footprint ~ -> Capacitors_SMD:c_0805
- C10: footprint ~ -> Capacitors_Tantalum_SMD:TantalC_SizeA_EIA-3216_HandSoldering
- D3, D4: footprint ~ -> LEDs:LED-0805
- R1, R10, R11, R12, R13, R14, R15, R16, R2, R3, R4, R5, R6, R7, R8, R9: footprint ~ -> Resistors_SMD:R_0805_HandSoldering

Commit message: MLS800 :  - assigning footprints
Parts:
- CON1: footprint (none) -> Connect:JACK_ALIM
- SW1: footprint ~ -> Discret:SW_PUSH
- X1: footprint ~ -> Crystals_Oscillators_SMD:Q_49U3HMS
- X2: footprint (none) -> Connect:USB_B
Changed lines of the file:
@@
 F 0 "CON1" H 1250 6350 60  0000 C CNN
 F 1 "BARREL_JACK" H 1250 5900 60  0000 C CNN
-F 2 "" H 1250 6100 60  0000 C CNN
+F 2 "Connect:JACK_ALIM" H 1250 6100 60  0001 C CNN
 F 3 "" H 1250 6100 60  0000 C CNN
 	1    1250 6100
@@
 F 0 "X1" H 1850 3700 60  0000 C CNN
 F 1 "16Mhz" H 1850 3400 60  0000 C CNN
-F 2 "~" H 1850 3550 60  0000 C CNN
+F 2 "Crystals_Oscillators_SMD:Q_49U3HMS" H 1850 3550 60  0001 C CNN
 F 3 "~" H 1850 3550 60  0000 C CNN
 	1    1850 3550
@@
 F 0 "SW1" H 1350 1560 50  0000 C CNN
 F 1 "SW_PUSH" H 1200 1370 50  0000 C CNN
-F 2 "~" H 1200 1450 60  0000 C CNN
+F 2 "Discret:SW_PUSH" H 1200 1450 60  0001 C CNN
 F 3 "~" H 1200 1450 60  0000 C CNN
 	1    1200 1450
@@
 F 0 "X2" H 4900 6000 60  0000 C CNN
 F 1 "USBMICRO" H 4950 6650 60  0000 C CNN
-F 2 "" H 4900 6300 60  0000 C CNN
+F 2 "Connect:USB_B" H 4900 6300 60  0000 C CNN
 F 3 "" H 4900 6300 60  0000 C CNN
 	1    4900 6300

Commit message: MLS800 :  - assigning footprints
Parts:
- removed X2: USBMICRO, Connect:USB_B, symbol USBMICRO
- added C12: 100nF, Capacitors_SMD:c_0805, symbol C
- added J1: USB, Connect:USB_B, symbol USB
- added VR1, VR2: CG0603MLC-05E, SMD_Packages:SMD-0603, symbol VR
- D1, D5: footprint ~ -> Imported:SOD-123
- D2: footprint ~ -> Diodes_SMD:Diode-SMB_Handsoldering
- F1: value FUSE -> MS-MSMF050-2; footprint ~ -> SMD_Packages:SMD-1812
- FB1: footprint ~ -> SMD_Packages:SMD-0805
- IC1: footprint DIP8 -> SMD_Packages:DIP-8_SMD
- P2: renamed from P1; footprint (none) -> Imported:DIN_5
- P3: renamed from P2; footprint (none) -> Imported:DIN_5
- SW1: footprint Discret:SW_PUSH -> ~
- U1: footprint ~ -> SMD_Packages:SOT-223
- U2: footprint (none) -> Housings_QFP:lqfp44
- U3: footprint (none) -> Housings_SOIC:SOIC-8_N
- renumbered P3 to P1, R12 to R10, R13 to R11, R5 to R12, R4 to R13, R16 to R15, R15 to R16, R6 to R4, R7 to R5, R8 to R6, R9 to R7, R10 to R8, R11 to R9
Connections:
- net D+: now also R12.2; no longer R12.1
- net D-: now also R13.2; no longer R13.1
- net DGND: now also J1.4 (GND), J1.5 (Shield_1), J1.6 (Shield_2), VR1.1, VR2.1
- net RX: now also C12.1
- net VCC: now also C12.2
- net at C10.1, F1.2: now also J1.1 (Vbus)
- new net: J1.2 (D-), R13.1, VR2.2
- new net: J1.3 (D+), R12.1, VR1.2
- no-connect marks 22 -> 21
Other:
- moved on the sheet: R12, R13, R16, U3
