File: mls800.sch (KiCad schematic (older format))
At the start: 50 parts, among them CON1 BARREL_JACK, IC1 6N137, J1 USB, P1 CONN_02X03, P2 DIN_5, P3 DIN_5, SW1 SW_PUSH, SW2 SW_TACT_LED_2, SW3 SW_TACT_LED_2, U1 LM340-5.0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

Commit message: MLS800 : created custom librairies
Connections:
- wire segments 120 -> 156
Changed lines of the file:
@@
 LIBS:contrib
 LIBS:valves
+LIBS:custom-i2c
+LIBS:custom-opto
+LIBS:custom-conn
+LIBS:custom-device
 LIBS:mls800-cache
 EELAYER 24 0
@@
 $Descr A4 11693 8268
 encoding utf-8
-Sheet 1 4
+Sheet 1 5
 Title ""
 Date "18 aug 2014"
@@
 P 4350 5900
 F 0 "F1" H 4450 5950 40  0000 C CNN
-F 1 "MS-MSMF050-2" H 4250 5850 40  0000 C CNN
+F 1 "MS-MSMF050-2" H 4250 5800 40  0000 C CNN
 F 2 "SMD_Packages:SMD-1812" H 4350 5900 60  0001 C CNN
 F 3 "~" H 4350 5900 60  0000 C CNN
@@
 	10350 1900 10350 1700
 Wire Wire Line
-	10350 2200 10950 2200
+	10350 2200 10550 2200
+Wire Wire Line
+	10550 2200 10750 2200
+Wire Wire Line
+	10750 2200 10950 2200
 Wire Wire Line
 	9500 1850 9350 1850
@@
 	6150 2600 5300 2600
 Wire Wire Line
-	6450 3600 6450 4000
+	6450 3600 6450 3850
+Wire Wire Line
+	6450 3850 6450 4000
 Wire Wire Line
 	5450 4000 5450 3850
@@
 	2500 2500 2850 2500
 Wire Wire Line
-	7050 5750 7150 5750
+	7050 5750 7100 5750
+Wire Wire Line
+	7100 5750 7150 5750
 Wire Wire Line
 	7100 5650 7150 5650
@@
 	2400 1350 2400 1450
 Wire Wire Line
-	2250 1350 2550 1350
+	2250 1350 2400 1350
+Wire Wire Line
+	2400 1350 2550 1350
 Connection ~ 2750 4500
 Wire Wire Line
@@
 	2750 4200 2850 4200
 Wire Wire Line
-	2450 4000 2850 4000
-Wire Wire Line
-	2750 4000 2750 4600
+	2450 4000 2750 4000
+Wire Wire Line
+	2750 4000 2850 4000
+Wire Wire Line
+	2750 4000 2750 4200
+Wire Wire Line
+	2750 4200 2750 4300
+Wire Wire Line
+	2750 4300 2750 4400
+Wire Wire Line
+	2750 4400 2750 4500
+Wire Wire Line
+	2750 4500 2750 4600
 Connection ~ 2650 2200
 Wire Wire Line
@@
 	5200 5350 5200 5400
 Wire Wire Line
-	4600 5350 5200 5350
-Wire Wire Line
-	4600 5300 4600 5400
+	4600 5350 4900 5350
+Wire Wire Line
+	4900 5350 5200 5350
+Wire Wire Line
+	4600 5300 4600 5350
+Wire Wire Line
+	4600 5350 4600 5400
 Connection ~ 4600 5900
 Wire Wire Line
-	4600 5800 4600 6550
+	4600 5800 4600 5900
+Wire Wire Line
+	4600 5900 4600 6550
 Wire Wire Line
 	2150 3700 2850 3700
@@
 	5300 2600 5300 2400
 Wire Wire Line
-	1700 950  2550 950
+	1700 950  2000 950
+Wire Wire Line
+	2000 950  2250 950
+Wire Wire Line
+	2250 950  2550 950
 Connection ~ 2000 950
 Connection ~ 2250 950
 Wire Wire Line
-	1500 1450 2000 1450
+	1500 1450 1700 1450
+Wire Wire Line
+	1700 1450 2000 1450
 Connection ~ 1700 1450
 Wire Wire Line
-	1700 6400 2750 6400
+	1700 6400 1950 6400
+Wire Wire Line
+	1950 6400 2350 6400
+Wire Wire Line
+	2350 6400 2750 6400
 Connection ~ 2900 6000
 Wire Wire Line
-	2750 6000 3050 6000
+	2750 6000 2900 6000
+Wire Wire Line
+	2900 6000 3050 6000
 Wire Wire Line
 	2150 3400 2850 3400
@@
 	2150 3850 2150 3700
 Wire Wire Line
-	2450 3000 2450 4000
+	2450 3000 2450 3200
+Wire Wire Line
+	2450 3200 2450 4000
 Connection ~ 2750 4000
 Connection ~ 2450 3200
 Wire Wire Line
-	2650 2100 2650 2300
-Wire Wire Line
-	5200 5800 5600 5800
+	2650 2100 2650 2200
+Wire Wire Line
+	2650 2200 2650 2300
+Wire Wire Line
+	5200 5800 5400 5800
+Wire Wire Line
+	5400 5800 5600 5800
 Connection ~ 5400 5800
 Wire Wire Line
@@
 	6150 3250 6150 3150
 Wire Wire Line
-	2350 6300 2350 6750
+	2350 6300 2350 6400
+Wire Wire Line
+	2350 6400 2350 6550
+Wire Wire Line
+	2350 6550 2350 6750
 Wire Wire Line
 	2350 6550 2400 6550
 Wire Wire Line
-	2200 6750 2500 6750
+	2200 6750 2350 6750
+Wire Wire Line
+	2350 6750 2500 6750
 Connection ~ 2350 6750
 Connection ~ 2350 6550
@@
 Connection ~ 1950 6400
 Wire Wire Line
-	2200 7250 2200 7450
+	2200 7250 2200 7350
+Wire Wire Line
+	2200 7350 2200 7450
 Connection ~ 2200 7350
 Wire Wire Line
-	2500 7250 2500 7450
+	2500 7250 2500 7350
+Wire Wire Line
+	2500 7350 2500 7450
 Connection ~ 2500 7350
 Wire Wire Line
@@
 	5050 3400 4750 3400
 Wire Wire Line
-	4350 6700 4600 6700
-Wire Wire Line
-	5350 6700 5850 6700
+	4350 6700 4500 6700
+Wire Wire Line
+	4500 6700 4600 6700
+Wire Wire Line
+	5350 6700 5750 6700
+Wire Wire Line
+	5750 6700 5850 6700
 Wire Wire Line
 	6350 6700 6600 6700
@@
 	6600 6550 6350 6550
 Wire Wire Line
-	5350 6550 5850 6550
-Wire Wire Line
-	7100 5650 7100 5850
+	5350 6550 5500 6550
+Wire Wire Line
+	5500 6550 5850 6550
+Wire Wire Line
+	7100 5650 7100 5750
+Wire Wire Line
+	7100 5750 7100 5850
 Connection ~ 7100 5750
 Wire Wire Line
@@
 	5350 6800 5350 7250
 Wire Wire Line
-	4600 7250 5750 7250
+	4600 7250 5350 7250
+Wire Wire Line
+	5350 7250 5500 7250
+Wire Wire Line
+	5500 7250 5750 7250
 Connection ~ 5500 7250
 Connection ~ 5350 7250
@@
 Connection ~ 10550 2200
 Wire Wire Line
-	10350 1700 10750 1700
+	10350 1700 10550 1700
+Wire Wire Line
+	10550 1700 10750 1700
 Connection ~ 10550 1700
+$Sheet
+S 8450 3900 1050 700
+U 543C4BC4
+F0 "Front panel" 60
+F1 "mls800_front_panel.sch" 60
+F2 "SDA" I L 8450 4000 60
+F3 "SCL" I L 8450 4150 60
+$EndSheet
+Wire Wire Line
+	8450 4000 8250 4000
+Wire Wire Line
+	8450 4150 8250 4150
+Text Label 8250 4150 0    60   ~ 0
+SCL
+Text Label 8250 4000 0    60   ~ 0
+SDA
 $EndSCHEMATC

Commit message: MLS800 : added LTC-5723HR  to custom-display library
MLS800 : fixed AS1115 pin placement to match main grid
Connections:
- net labels added: UIINT
- wire segments 156 -> 123
Changed lines of the file:
@@
 LIBS:custom-conn
 LIBS:custom-device
+LIBS:custom-display
 LIBS:mls800-cache
 EELAYER 24 0
@@
 	10350 1900 10350 1700
 Wire Wire Line
-	10350 2200 10550 2200
-Wire Wire Line
-	10550 2200 10750 2200
-Wire Wire Line
-	10750 2200 10950 2200
+	10350 2200 10950 2200
 Wire Wire Line
 	9500 1850 9350 1850
@@
 	6150 2600 5300 2600
 Wire Wire Line
-	6450 3600 6450 3850
-Wire Wire Line
-	6450 3850 6450 4000
+	6450 3600 6450 4000
 Wire Wire Line
 	5450 4000 5450 3850
@@
 	2500 2500 2850 2500
 Wire Wire Line
-	7050 5750 7100 5750
-Wire Wire Line
-	7100 5750 7150 5750
+	7050 5750 7150 5750
 Wire Wire Line
 	7100 5650 7150 5650
@@
 	2400 1350 2400 1450
 Wire Wire Line
-	2250 1350 2400 1350
-Wire Wire Line
-	2400 1350 2550 1350
+	2250 1350 2550 1350
 Connection ~ 2750 4500
 Wire Wire Line
@@
 	2750 4200 2850 4200
 Wire Wire Line
-	2450 4000 2750 4000
-Wire Wire Line
-	2750 4000 2850 4000
-Wire Wire Line
-	2750 4000 2750 4200
-Wire Wire Line
-	2750 4200 2750 4300
-Wire Wire Line
-	2750 4300 2750 4400
-Wire Wire Line
-	2750 4400 2750 4500
-Wire Wire Line
-	2750 4500 2750 4600
+	2450 4000 2850 4000
+Wire Wire Line
+	2750 4000 2750 4600
 Connection ~ 2650 2200
 Wire Wire Line
@@
 	5200 5350 5200 5400
 Wire Wire Line
-	4600 5350 4900 5350
-Wire Wire Line
-	4900 5350 5200 5350
-Wire Wire Line
-	4600 5300 4600 5350
-Wire Wire Line
-	4600 5350 4600 5400
+	4600 5350 5200 5350
+Wire Wire Line
+	4600 5300 4600 5400
 Connection ~ 4600 5900
 Wire Wire Line
-	4600 5800 4600 5900
-Wire Wire Line
-	4600 5900 4600 6550
+	4600 5800 4600 6550
 Wire Wire Line
 	2150 3700 2850 3700
@@
 	5300 2600 5300 2400
 Wire Wire Line
-	1700 950  2000 950
-Wire Wire Line
-	2000 950  2250 950
-Wire Wire Line
-	2250 950  2550 950
+	1700 950  2550 950
 Connection ~ 2000 950
 Connection ~ 2250 950
 Wire Wire Line
-	1500 1450 1700 1450
-Wire Wire Line
-	1700 1450 2000 1450
+	1500 1450 2000 1450
 Connection ~ 1700 1450
 Wire Wire Line
-	1700 6400 1950 6400
-Wire Wire Line
-	1950 6400 2350 6400
-Wire Wire Line
-	2350 6400 2750 6400
+	1700 6400 2750 6400
 Connection ~ 2900 6000
 Wire Wire Line
-	2750 6000 2900 6000
-Wire Wire Line
-	2900 6000 3050 6000
+	2750 6000 3050 6000
 Wire Wire Line
 	2150 3400 2850 3400
@@
 	2150 3850 2150 3700
 Wire Wire Line
-	2450 3000 2450 3200
-Wire Wire Line
-	2450 3200 2450 4000
+	2450 3000 2450 4000
 Connection ~ 2750 4000
 Connection ~ 2450 3200
 Wire Wire Line
-	2650 2100 2650 2200
-Wire Wire Line
-	2650 2200 2650 2300
-Wire Wire Line
-	5200 5800 5400 5800
-Wire Wire Line
-	5400 5800 5600 5800
+	2650 2100 2650 2300
+Wire Wire Line
+	5200 5800 5600 5800
 Connection ~ 5400 5800
 Wire Wire Line
@@
 	6150 3250 6150 3150
 Wire Wire Line
-	2350 6300 2350 6400
-Wire Wire Line
-	2350 6400 2350 6550
-Wire Wire Line
-	2350 6550 2350 6750
+	2350 6300 2350 6750
 Wire Wire Line
 	2350 6550 2400 6550
 Wire Wire Line
-	2200 6750 2350 6750
-Wire Wire Line
-	2350 6750 2500 6750
+	2200 6750 2500 6750
 Connection ~ 2350 6750
 Connection ~ 2350 6550
@@
 Connection ~ 1950 6400
 Wire Wire Line
-	2200 7250 2200 7350
-Wire Wire Line
-	2200 7350 2200 7450
+	2200 7250 2200 7450
 Connection ~ 2200 7350
 Wire Wire Line
-	2500 7250 2500 7350
-Wire Wire Line
-	2500 7350 2500 7450
+	2500 7250 2500 7450
 Connection ~ 2500 7350
 Wire Wire Line
@@
 	5050 3400 4750 3400
 Wire Wire Line
-	4350 6700 4500 6700
-Wire Wire Line
-	4500 6700 4600 6700
-Wire Wire Line
-	5350 6700 5750 6700
-Wire Wire Line
-	5750 6700 5850 6700
+	4350 6700 4600 6700
+Wire Wire Line
+	5350 6700 5850 6700
 Wire Wire Line
 	6350 6700 6600 6700
@@
 	6600 6550 6350 6550
 Wire Wire Line
-	5350 6550 5500 6550
-Wire Wire Line
-	5500 6550 5850 6550
-Wire Wire Line
-	7100 5650 7100 5750
-Wire Wire Line
-	7100 5750 7100 5850
+	5350 6550 5850 6550
+Wire Wire Line
+	7100 5650 7100 5850
 Connection ~ 7100 5750
 Wire Wire Line
@@
 	5350 6800 5350 7250
 Wire Wire Line
-	4600 7250 5350 7250
-Wire Wire Line
-	5350 7250 5500 7250
-Wire Wire Line
-	5500 7250 5750 7250
+	4600 7250 5750 7250
 Connection ~ 5500 7250
 Connection ~ 5350 7250
@@
 Connection ~ 10550 2200
 Wire Wire Line
-	10350 1700 10550 1700
-Wire Wire Line
-	10550 1700 10750 1700
+	10350 1700 10750 1700
 Connection ~ 10550 1700
+Wire Wire Line
+	7850 3250 7650 3250
+Wire Wire Line
+	7850 3400 7650 3400
+Text Label 7650 3400 0    60   ~ 0
+SCL
+Text Label 7650 3250 0    60   ~ 0
+SDA
 $Sheet
-S 8450 3900 1050 700
+S 7850 3150 1050 700
 U 543C4BC4
 F0 "Front panel" 60
 F1 "mls800_front_panel.sch" 60
-F2 "SDA" I L 8450 4000 60
-F3 "SCL" I L 8450 4150 60
+F2 "SDA" I L 7850 3250 60
+F3 "SCL" I L 7850 3400 60
+F4 "IRQ" I L 7850 3550 60
 $EndSheet
-Wire Wire Line
-	8450 4000 8250 4000
-Wire Wire Line
-	8450 4150 8250 4150
-Text Label 8250 4150 0    60   ~ 0
-SCL
-Text Label 8250 4000 0    60   ~ 0
-SDA
+Text Label 7600 3550 0    60   ~ 0
+UIINT
+Wire Wire Line
+	7600 3550 7850 3550
 $EndSCHEMATC

Commit message: MLS800 : fixed missing components
Parts:
- SW2, SW3: value SW_TACT_LED_2 -> SW_TACT_LED; symbol SW_TACT_LED_2 -> SW_TACT_LED
Changed lines of the file:
@@
 LIBS:custom-device
 LIBS:custom-display
+LIBS:custom-micro
 LIBS:mls800-cache
 EELAYER 24 0
@@
 RXLED
 $Comp
-L SW_TACT_LED_2 SW2
+L SW_TACT_LED SW2
 U 2 1 53B9C16B
 P 6450 2700
 F 0 "SW2" H 6550 2600 60  0000 C CNN
-F 1 "SW_TACT_LED_2" H 6500 2600 60  0001 C CNN
+F 1 "SW_TACT_LED" H 6500 2600 60  0001 C CNN
 F 2 "" H 6450 2700 60  0000 C CNN
 F 3 "" H 6450 2700 60  0000 C CNN
@@
 $EndComp
 $Comp
-L SW_TACT_LED_2 SW2
+L SW_TACT_LED SW2
 U 1 1 53B9C171
 P 6450 2500
 F 0 "SW2" H 6550 2650 60  0000 C CNN
-F 1 "SW_TACT_LED_2" H 6500 2400 60  0001 C CNN
+F 1 "SW_TACT_LED" H 6500 2400 60  0001 C CNN
 F 2 "" H 6450 2500 60  0000 C CNN
 F 3 "" H 6450 2500 60  0000 C CNN
@@
 $EndComp
 $Comp
-L SW_TACT_LED_2 SW3
+L SW_TACT_LED SW3
 U 2 1 53B9C18C
 P 6450 3250
 F 0 "SW3" H 6550 3150 60  0000 C CNN
-F 1 "SW_TACT_LED_2" H 6500 3150 60  0001 C CNN
+F 1 "SW_TACT_LED" H 6500 3150 60  0001 C CNN
 F 2 "" H 6450 3250 60  0000 C CNN
 F 3 "" H 6450 3250 60  0000 C CNN
@@
 $EndComp
 $Comp
-L SW_TACT_LED_2 SW3
+L SW_TACT_LED SW3
 U 1 1 53B9C192
 P 6450 3050
 F 0 "SW3" H 6550 3200 60  0000 C CNN
-F 1 "SW_TACT_LED_2" H 6500 2950 60  0001 C CNN
+F 1 "SW_TACT_LED" H 6500 2950 60  0001 C CNN
 F 2 "" H 6450 3050 60  0000 C CNN
 F 3 "" H 6450 3050 60  0000 C CNN

Commit message: MLS800 : fixed broken layout
MLS800 : added some comments on schematics rather than using a notepad :)
Other:
- note added: "Do not forget restistances on SDA & SCL lines !"
Changed lines of the file:
@@
 Wire Wire Line
 	7600 3550 7850 3550
+Text Notes 5650 4550 0    60   ~ 0
+Do not forget restistances on SDA & SCL lines !
 $EndSCHEMATC

Commit message: MLS800 : disabled switch tact led "interchangeable" units => fixed annotations
MLS800 : front panel schematic seems to be completed
Connections:
- net DGND: now also SW2.2, SW3.2; no longer SW2.1, SW3.1
- net EDIT: now also SW2.4; no longer SW2.3
- net EXIT: now also SW3.4; no longer SW3.3
- net UI INT: no longer U2.28 (PB4(ADC11))
- net VCC: now also SW2.1, SW3.1; no longer SW2.2, SW3.2
- net at R10.1: now also SW3.3; no longer SW3.4
- net at R8.1: now also SW2.3; no longer SW2.4
- new net UI_INT: U2.28 (PB4(ADC11))

Commit message: MLS800 : disabled switch tact led "interchangeable" units => fixed annotations
MLS800 : fixed some erc errors in old "misc" sheet
Connections:
- no-connect marks 21 -> 22
Changed lines of the file:
@@
 $EndComp
 $Comp
-L GND #PWR11
+L GND #PWR01
 U 1 1 53505891
 P 2400 6550
-F 0 "#PWR11" H 2400 6550 30  0001 C CNN
+F 0 "#PWR01" H 2400 6550 30  0001 C CNN
 F 1 "GND" H 2400 6480 30  0001 C CNN
 F 2 "" H 2400 6550 60  0000 C CNN
@@
 POWER\n
 $Comp
-L VCC #PWR13
+L VCC #PWR02
 U 1 1 53505C75
 P 2650 2100
-F 0 "#PWR13" H 2650 2200 30  0001 C CNN
+F 0 "#PWR02" H 2650 2200 30  0001 C CNN
 F 1 "VCC" H 2650 2200 30  0000 C CNN
 F 2 "" H 2650 2100 60  0000 C CNN
@@
 $EndComp
 $Comp
-L VCC #PWR6
+L VCC #PWR03
 U 1 1 535068DE
 P 2000 950
-F 0 "#PWR6" H 2000 1050 30  0001 C CNN
+F 0 "#PWR03" H 2000 1050 30  0001 C CNN
 F 1 "VCC" H 2000 1050 30  0000 C CNN
 F 2 "" H 2000 950 60  0000 C CNN
@@
 $EndComp
 $Comp
-L VCC #PWR7
+L VCC #PWR04
 U 1 1 5350782A
 P 2000 4450
-F 0 "#PWR7" H 2000 4550 30  0001 C CNN
+F 0 "#PWR04" H 2000 4550 30  0001 C CNN
 F 1 "VCC" H 2000 4550 30  0000 C CNN
 F 2 "" H 2000 4450 60  0000 C CNN
@@
 Text Label 9850 3600 0    59   ~ 0
 SCL
-Text Label 9750 3750 0    59   ~ 0
-UI INT
 Text Label 9850 4550 0    59   ~ 0
 SDA
@@
 $EndComp
 $Comp
-L VCC #PWR29
+L VCC #PWR05
 U 1 1 53A795F5
 P 6650 3250
-F 0 "#PWR29" H 6650 3350 30  0001 C CNN
+F 0 "#PWR05" H 6650 3350 30  0001 C CNN
 F 1 "VCC" H 6650 3350 30  0000 C CNN
 F 2 "" H 6650 3250 60  0000 C CNN
@@
 F2 "SDA" I L 10050 3450 60
 F3 "SCL" I L 10050 3600 60
-F4 "UI INT" I L 10050 3750 60
+F4 "UI_INT" I L 10050 3750 60
 $EndSheet
 Text GLabel 8550 5950 2    28   Input ~ 0
@@
 SDA
 $Comp
-L VCC #PWR31
+L VCC #PWR06
 U 1 1 53A7B7A6
 P 7850 5350
-F 0 "#PWR31" H 7850 5450 30  0001 C CNN
+F 0 "#PWR06" H 7850 5450 30  0001 C CNN
 F 1 "VCC" H 7850 5450 30  0000 C CNN
 F 2 "" H 7850 5350 60  0000 C CNN
@@
 $EndComp
 $Comp
-L VCC #PWR4
+L VCC #PWR07
 U 1 1 53A7C589
 P 1800 2500
-F 0 "#PWR4" H 1800 2600 30  0001 C CNN
+F 0 "#PWR07" H 1800 2600 30  0001 C CNN
 F 1 "VCC" H 1800 2600 30  0000 C CNN
 F 2 "" H 1800 2500 60  0000 C CNN
@@
 $EndComp
 $Comp
-L VCC #PWR22
+L VCC #PWR08
 U 1 1 53A8C536
 P 5650 3050
-F 0 "#PWR22" H 5650 3150 30  0001 C CNN
+F 0 "#PWR08" H 5650 3150 30  0001 C CNN
 F 1 "VCC" H 5650 3150 30  0000 C CNN
 F 2 "" H 5650 3050 60  0000 C CNN
@@
 $EndComp
 $Comp
-L VCC #PWR27
+L VCC #PWR09
 U 1 1 53A8D128
 P 6650 2700
-F 0 "#PWR27" H 6650 2800 30  0001 C CNN
+F 0 "#PWR09" H 6650 2800 30  0001 C CNN
 F 1 "VCC" H 6650 2800 30  0000 C CNN
 F 2 "" H 6650 2700 60  0000 C CNN
@@
 $EndComp
 $Comp
-L VCC #PWR35
+L VCC #PWR010
 U 1 1 53A8E22E
 P 10750 1700
-F 0 "#PWR35" H 10750 1800 30  0001 C CNN
+F 0 "#PWR010" H 10750 1800 30  0001 C CNN
 F 1 "VCC" H 10750 1800 30  0000 C CNN
 F 2 "" H 10750 1700 60  0000 C CNN
@@
 $EndComp
 $Comp
-L VCC #PWR36
+L VCC #PWR011
 U 1 1 53A8E259
 P 10800 1100
-F 0 "#PWR36" H 10800 1200 30  0001 C CNN
+F 0 "#PWR011" H 10800 1200 30  0001 C CNN
 F 1 "VCC" H 10800 1200 30  0000 C CNN
 F 2 "" H 10800 1100 60  0000 C CNN
@@
 $EndSheet
 $Comp
-L PWR_FLAG #FLG5
+L PWR_FLAG #FLG012
 U 1 1 53A950B6
 P 5600 5800
-F 0 "#FLG5" H 5600 5895 30  0001 C CNN
+F 0 "#FLG012" H 5600 5895 30  0001 C CNN
 F 1 "PWR_FLAG" H 5600 5980 30  0000 C CNN
 F 2 "" H 5600 5800 60  0000 C CNN
@@
 $EndComp
 $Comp
-L DGND #PWR25
+L DGND #PWR013
 U 1 1 53F1874E
 P 6450 4000
-F 0 "#PWR25" H 6450 4000 40  0001 C CNN
+F 0 "#PWR013" H 6450 4000 40  0001 C CNN
 F 1 "DGND" H 6450 3930 40  0000 C CNN
 F 2 "" H 6450 4000 60  0000 C CNN
@@
 $EndComp
 $Comp
-L DGND #PWR26
+L DGND #PWR014
 U 1 1 53F18858
 P 6650 2500
-F 0 "#PWR26" H 6650 2500 40  0001 C CNN
+F 0 "#PWR014" H 6650 2500 40  0001 C CNN
 F 1 "DGND" H 6650 2430 40  0000 C CNN
 F 2 "" H 6650 2500 60  0000 C CNN
@@
 $EndComp
 $Comp
-L DGND #PWR30
+L DGND #PWR015
 U 1 1 53F18B44
 P 7050 5750
-F 0 "#PWR30" H 7050 5750 40  0001 C CNN
+F 0 "#PWR015" H 7050 5750 40  0001 C CNN
 F 1 "DGND" H 7050 5680 40  0000 C CNN
 F 2 "" H 7050 5750 60  0000 C CNN
@@
 $EndComp
 $Comp
-L DGND #PWR32
+L DGND #PWR016
 U 1 1 53F18C26
 P 7850 6350
-F 0 "#PWR32" H 7850 6350 40  0001 C CNN
+F 0 "#PWR016" H 7850 6350 40  0001 C CNN
 F 1 "DGND" H 7850 6280 40  0000 C CNN
 F 2 "" H 7850 6350 60  0000 C CNN
@@
 $EndComp
 $Comp
-L DGND #PWR34
+L DGND #PWR017
 U 1 1 53F18CDE
 P 10200 2200
-F 0 "#PWR34" H 10200 2200 40  0001 C CNN
+F 0 "#PWR017" H 10200 2200 40  0001 C CNN
 F 1 "DGND" H 10200 2130 40  0000 C CNN
 F 2 "" H 10200 2200 60  0000 C CNN
@@
 $EndComp
 $Comp
-L DGND #PWR33
+L DGND #PWR018
 U 1 1 53F18FB8
 P 9700 700
-F 0 "#PWR33" H 9700 700 40  0001 C CNN
+F 0 "#PWR018" H 9700 700 40  0001 C CNN
 F 1 "DGND" H 9700 630 40  0000 C CNN
 F 2 "" H 9700 700 60  0000 C CNN
@@
 $EndComp
 $Comp
-L DGND #PWR24
+L DGND #PWR019
 U 1 1 53F19196
 P 6150 2300
-F 0 "#PWR24" H 6150 2300 40  0001 C CNN
+F 0 "#PWR019" H 6150 2300 40  0001 C CNN
 F 1 "DGND" H 6150 2230 40  0000 C CNN
 F 2 "" H 6150 2300 60  0000 C CNN
@@
 $EndComp
 $Comp
-L DGND #PWR14
+L DGND #PWR020
 U 1 1 53F191E5
 P 2750 4600
-F 0 "#PWR14" H 2750 4600 40  0001 C CNN
+F 0 "#PWR020" H 2750 4600 40  0001 C CNN
 F 1 "DGND" H 2750 4530 40  0000 C CNN
 F 2 "" H 2750 4600 60  0000 C CNN
@@
 $EndComp
 $Comp
-L DGND #PWR8
+L DGND #PWR021
 U 1 1 53F193C3
 P 2000 4650
-F 0 "#PWR8" H 2000 4650 40  0001 C CNN
+F 0 "#PWR021" H 2000 4650 40  0001 C CNN
 F 1 "DGND" H 2000 4580 40  0000 C CNN
 F 2 "" H 2000 4650 60  0000 C CNN
@@
 $EndComp
 $Comp
-L DGND #PWR18
+L DGND #PWR022
 U 1 1 53F19742
 P 4350 6700
-F 0 "#PWR18" H 4350 6700 40  0001 C CNN
+F 0 "#PWR022" H 4350 6700 40  0001 C CNN
 F 1 "DGND" H 4350 6630 40  0000 C CNN
 F 2 "" H 4350 6700 60  0000 C CNN
@@
 $EndComp
 $Comp
-L DGND #PWR12
+L DGND #PWR023
 U 1 1 53F198E1
 P 2500 7450
-F 0 "#PWR12" H 2500 7450 40  0001 C CNN
+F 0 "#PWR023" H 2500 7450 40  0001 C CNN
 F 1 "DGND" H 2500 7380 40  0000 C CNN
 F 2 "" H 2500 7450 60  0000 C CNN
@@
 $EndComp
 $Comp
-L DGND #PWR23
+L DGND #PWR024
 U 1 1 53F19B2D
 P 5650 3250
-F 0 "#PWR23" H 5650 3250 40  0001 C CNN
+F 0 "#PWR024" H 5650 3250 40  0001 C CNN
 F 1 "DGND" H 5650 3180 40  0000 C CNN
 F 2 "" H 5650 3250 60  0000 C CNN
@@
 $EndComp
 $Comp
-L DGND #PWR21
+L DGND #PWR025
 U 1 1 53F19BC6
 P 5650 2700
-F 0 "#PWR21" H 5650 2700 40  0001 C CNN
+F 0 "#PWR025" H 5650 2700 40  0001 C CNN
 F 1 "DGND" H 5650 2630 40  0000 C CNN
 F 2 "" H 5650 2700 60  0000 C CNN
@@
 $EndComp
 $Comp
-L AGND #PWR9
+L AGND #PWR026
 U 1 1 53F1A7A7
 P 2200 7450
-F 0 "#PWR9" H 2200 7450 40  0001 C CNN
+F 0 "#PWR026" H 2200 7450 40  0001 C CNN
 F 1 "AGND" H 2200 7380 50  0000 C CNN
 F 2 "" H 2200 7450 60  0000 C CNN
@@
 $EndComp
 $Comp
-L DGND #PWR2
+L DGND #PWR027
 U 1 1 53F1C7D0
 P 1450 3250
-F 0 "#PWR2" H 1450 3250 40  0001 C CNN
+F 0 "#PWR027" H 1450 3250 40  0001 C CNN
 F 1 "DGND" H 1450 3180 40  0000 C CNN
 F 2 "" H 1450 3250 60  0000 C CNN
@@
 $EndComp
 $Comp
-L DGND #PWR3
+L DGND #PWR028
 U 1 1 53F1C800
 P 1450 3850
-F 0 "#PWR3" H 1450 3850 40  0001 C CNN
+F 0 "#PWR028" H 1450 3850 40  0001 C CNN
 F 1 "DGND" H 1450 3780 40  0000 C CNN
 F 2 "" H 1450 3850 60  0000 C CNN
@@
 $EndComp
 $Comp
-L DGND #PWR5
+L DGND #PWR029
 U 1 1 53F1C810
 P 1850 2800
-F 0 "#PWR5" H 1850 2800 40  0001 C CNN
+F 0 "#PWR029" H 1850 2800 40  0001 C CNN
 F 1 "DGND" H 1850 2730 40  0000 C CNN
 F 2 "" H 1850 2800 60  0000 C CNN
@@
 $EndComp
 $Comp
-L DGND #PWR1
+L DGND #PWR030
 U 1 1 53F1C84A
 P 900 1450
-F 0 "#PWR1" H 900 1450 40  0001 C CNN
+F 0 "#PWR030" H 900 1450 40  0001 C CNN
 F 1 "DGND" H 900 1380 40  0000 C CNN
 F 2 "" H 900 1450 60  0000 C CNN
@@
 $EndComp
 $Comp
-L DGND #PWR10
+L DGND #PWR031
 U 1 1 53F1C8D8
 P 2400 1450
-F 0 "#PWR10" H 2400 1450 40  0001 C CNN
+F 0 "#PWR031" H 2400 1450 40  0001 C CNN
 F 1 "DGND" H 2400 1380 40  0000 C CNN
 F 2 "" H 2400 1450 60  0000 C CNN
@@
 $EndComp
 $Comp
-L PWR_FLAG #FLG1
+L PWR_FLAG #FLG032
 U 1 1 53F1D218
 P 2200 7350
-F 0 "#FLG1" H 2200 7445 30  0001 C CNN
+F 0 "#FLG032" H 2200 7445 30  0001 C CNN
 F 1 "PWR_FLAG" H 2200 7530 30  0000 C CNN
 F 2 "" H 2200 7350 60  0000 C CNN
@@
 $EndComp
 $Comp
-L PWR_FLAG #FLG3
+L PWR_FLAG #FLG033
 U 1 1 53F1D28F
 P 2500 7350
-F 0 "#FLG3" H 2500 7445 30  0001 C CNN
+F 0 "#FLG033" H 2500 7445 30  0001 C CNN
 F 1 "PWR_FLAG" H 2500 7530 30  0000 C CNN
 F 2 "" H 2500 7350 60  0000 C CNN
@@
 $EndComp
 $Comp
-L DGND #PWR19
+L DGND #PWR034
 U 1 1 53F1D8FC
 P 4600 5300
-F 0 "#PWR19" H 4600 5300 40  0001 C CNN
+F 0 "#PWR034" H 4600 5300 40  0001 C CNN
 F 1 "DGND" H 4600 5230 40  0000 C CNN
 F 2 "" H 4600 5300 60  0000 C CNN
@@
 $EndComp
 $Comp
-L DGND #PWR28
+L DGND #PWR035
 U 1 1 53F1D962
 P 6650 3050
-F 0 "#PWR28" H 6650 3050 40  0001 C CNN
+F 0 "#PWR035" H 6650 3050 40  0001 C CNN
 F 1 "DGND" H 6650 2980 40  0000 C CNN
 F 2 "" H 6650 3050 60  0000 C CNN
@@
 $EndComp
 $Comp
-L PWR_FLAG #FLG2
+L PWR_FLAG #FLG036
 U 1 1 53F1D998
 P 2350 6550
-F 0 "#FLG2" H 2350 6645 30  0001 C CNN
+F 0 "#FLG036" H 2350 6645 30  0001 C CNN
 F 1 "PWR_FLAG" H 2350 6730 30  0000 C CNN
 F 2 "" H 2350 6550 60  0000 C CNN
@@
 $EndComp
 $Comp
-L PWR_FLAG #FLG4
+L PWR_FLAG #FLG037
 U 1 1 53F12BDD
 P 3050 6000
-F 0 "#FLG4" H 3050 6095 30  0001 C CNN
+F 0 "#FLG037" H 3050 6095 30  0001 C CNN
 F 1 "PWR_FLAG" H 3050 6180 30  0000 C CNN
 F 2 "" H 3050 6000 60  0000 C CNN
@@
 $EndComp
 $Comp
-L VCC #PWR16
+L VCC #PWR038
 U 1 1 53F12F8A
 P 2900 6000
-F 0 "#PWR16" H 2900 6100 30  0001 C CNN
+F 0 "#PWR038" H 2900 6100 30  0001 C CNN
 F 1 "VCC" H 2900 6100 30  0000 C CNN
 F 2 "" H 2900 6000 60  0000 C CNN
@@
 Wire Wire Line
 	6150 2700 6150 2600
+NoConn ~ 9750 3750
 $EndSCHEMATC

Commit message: MLS800 : removed useless power flag
MLS800 : fixed most errors and warnings
ATMEGA32U : fixed missing "power input" pins
Other:
- note added: "Aref should be connected to something else than GND.\nCheck datasheet at chatper 24.2 page 294"
Changed lines of the file:
@@
 $EndComp
 $Comp
-L PWR_FLAG #FLG037
-U 1 1 53F12BDD
-P 3050 6000
-F 0 "#FLG037" H 3050 6095 30  0001 C CNN
-F 1 "PWR_FLAG" H 3050 6180 30  0000 C CNN
-F 2 "" H 3050 6000 60  0000 C CNN
-F 3 "" H 3050 6000 60  0000 C CNN
-	1    3050 6000
-	1    0    0    -1
-$EndComp
-$Comp
-L VCC #PWR038
+L VCC #PWR037
 U 1 1 53F12F8A
 P 2900 6000
-F 0 "#PWR038" H 2900 6100 30  0001 C CNN
+F 0 "#PWR037" H 2900 6100 30  0001 C CNN
 F 1 "VCC" H 2900 6100 30  0000 C CNN
 F 2 "" H 2900 6000 60  0000 C CNN
@@
 Wire Wire Line
 	1700 6400 2750 6400
-Connection ~ 2900 6000
-Wire Wire Line
-	2750 6000 3050 6000
 Wire Wire Line
 	2150 3400 2850 3400
@@
 	6150 2700 6150 2600
 NoConn ~ 9750 3750
+Text Notes 2300 4900 0    60   ~ 0
+Aref should be connected to something else than GND.\nCheck datasheet at chatper 24.2 page 294
+Wire Wire Line
+	2900 6000 2750 6000
 $EndSCHEMATC
