File: mls800_display.sch (KiCad schematic (older format))
At the start: 9 parts

Commit message: MLS800  * Lots of change in diagram/schematic  * Added external parts
Parts:
- gave numbers to parts that had none: 9
Connections:
- wire segments 24 -> 25
Other:
- moved on the sheet: Q17, Q18
Changed lines of the file:
@@
 Sheet 3 4
 Title ""
-Date "18 may 2014"
+Date "23 jun 2014"
 Rev ""
 Comp ""
@@
 $EndDescr
 $Comp
-L SAA1064T IC?
+L SAA1064T IC2
 U 1 1 534730A9
 P 1500 2450
-F 0 "IC?" H 1200 3500 50  0000 L BNN
+F 0 "IC2" H 1200 3500 50  0000 L BNN
 F 1 "SAA1064T" H 1200 1250 50  0000 L BNN
 F 2 "micro-philips-SO24" H 1500 2600 50  0001 C CNN
@@
 	1    0    0    -1
 $EndComp
-Text GLabel 1100 2050 0    28   Input ~ 0
-SCL
-$Comp
-L VCC #PWR?
+$Comp
+L VCC #PWR111
 U 1 1 534730B8
 P 1100 1650
-F 0 "#PWR?" H 1100 1750 30  0001 C CNN
+F 0 "#PWR111" H 1100 1750 30  0001 C CNN
 F 1 "VCC" H 1100 1750 30  0000 C CNN
 F 2 "" H 1100 1650 60  0000 C CNN
@@
 $EndComp
 $Comp
-L GND #PWR?
+L GND #PWR113
 U 1 1 534730C7
 P 1100 3350
-F 0 "#PWR?" H 1100 3350 30  0001 C CNN
+F 0 "#PWR113" H 1100 3350 30  0001 C CNN
 F 1 "GND" H 1100 3280 30  0001 C CNN
 F 2 "" H 1100 3350 60  0000 C CNN
@@
 	0    1    1    0
 $EndComp
-Text GLabel 1100 2250 0    28   Input ~ 0
-SDA
-$Comp
-L C C?
+$Comp
+L C C12
 U 1 1 534730D6
 P 900 2850
-F 0 "C?" H 900 2950 40  0000 L CNN
+F 0 "C12" H 900 2950 40  0000 L CNN
 F 1 "2.7nF" H 906 2765 40  0000 L CNN
 F 2 "~" H 938 2700 30  0000 C CNN
@@
 $EndComp
 $Comp
-L GND #PWR?
+L GND #PWR108
 U 1 1 534730F6
 P 700 2850
-F 0 "#PWR?" H 700 2850 30  0001 C CNN
+F 0 "#PWR108" H 700 2850 30  0001 C CNN
 F 1 "GND" H 700 2780 30  0001 C CNN
 F 2 "" H 700 2850 60  0000 C CNN
@@
 $EndComp
 $Comp
-L C C?
+L C C11
 U 1 1 534730FC
 P 800 2300
-F 0 "C?" H 800 2400 40  0000 L CNN
+F 0 "C11" H 800 2400 40  0000 L CNN
 F 1 "100nF" H 806 2215 40  0000 L CNN
 F 2 "~" H 838 2150 30  0000 C CNN
@@
 $EndComp
 $Comp
-L GND #PWR?
+L GND #PWR110
 U 1 1 53473118
 P 800 2500
-F 0 "#PWR?" H 800 2500 30  0001 C CNN
+F 0 "#PWR110" H 800 2500 30  0001 C CNN
 F 1 "GND" H 800 2430 30  0001 C CNN
 F 2 "" H 800 2500 60  0000 C CNN
@@
 $EndComp
 $Comp
-L VCC #PWR?
+L VCC #PWR109
 U 1 1 53473123
 P 800 2100
-F 0 "#PWR?" H 800 2200 30  0001 C CNN
+F 0 "#PWR109" H 800 2200 30  0001 C CNN
 F 1 "VCC" H 800 2200 30  0000 C CNN
 F 2 "" H 800 2100 60  0000 C CNN
@@
 $EndComp
 $Comp
-L NPN Q?
+L NPN Q18
 U 1 1 5347312B
-P 2000 3650
-F 0 "Q?" H 2000 3500 50  0000 R CNN
-F 1 "NPN" H 2000 3800 50  0000 R CNN
-F 2 "~" H 2000 3650 60  0000 C CNN
-F 3 "~" H 2000 3650 60  0000 C CNN
-	1    2000 3650
+P 2400 3650
+F 0 "Q18" H 2400 3500 50  0000 R CNN
+F 1 "NPN" H 2400 3800 50  0000 R CNN
+F 2 "~" H 2400 3650 60  0000 C CNN
+F 3 "~" H 2400 3650 60  0000 C CNN
+	1    2400 3650
 	0    1    1    0
 $EndComp
 $Comp
-L NPN Q?
+L NPN Q17
 U 1 1 53473138
-P 2000 1350
-F 0 "Q?" H 2000 1200 50  0000 R CNN
-F 1 "NPN" H 2000 1500 50  0000 R CNN
-F 2 "~" H 2000 1350 60  0000 C CNN
-F 3 "~" H 2000 1350 60  0000 C CNN
-	1    2000 1350
+P 2400 1350
+F 0 "Q17" H 2400 1200 50  0000 R CNN
+F 1 "NPN" H 2400 1500 50  0000 R CNN
+F 2 "~" H 2400 1350 60  0000 C CNN
+F 3 "~" H 2400 1350 60  0000 C CNN
+	1    2400 1350
 	0    -1   -1   0
 $EndComp
 $Comp
-L VCC #PWR?
+L VCC #PWR115
 U 1 1 5347313E
-P 2200 3750
-F 0 "#PWR?" H 2200 3850 30  0001 C CNN
-F 1 "VCC" H 2200 3850 30  0000 C CNN
-F 2 "" H 2200 3750 60  0000 C CNN
-F 3 "" H 2200 3750 60  0000 C CNN
-	1    2200 3750
+P 2600 3750
+F 0 "#PWR115" H 2600 3850 30  0001 C CNN
+F 1 "VCC" H 2600 3850 30  0000 C CNN
+F 2 "" H 2600 3750 60  0000 C CNN
+F 3 "" H 2600 3750 60  0000 C CNN
+	1    2600 3750
 	0    1    1    0
 $EndComp
 $Comp
-L 7SEGM S?
+L 7SEGM S3
 U 1 1 53473146
 P 4200 2500
-F 0 "S?" H 4200 3150 60  0000 C CNN
+F 0 "S3" H 4200 3150 60  0000 C CNN
 F 1 "7SEGM" H 4200 1850 60  0000 C CNN
 F 2 "~" H 4200 2500 60  0000 C CNN
@@
 $EndComp
 $Comp
-L 7SEGM S?
+L 7SEGM S4
 U 1 1 53473153
 P 5900 2500
-F 0 "S?" H 5900 3150 60  0000 C CNN
+F 0 "S4" H 5900 3150 60  0000 C CNN
 F 1 "7SEGM" H 5900 1850 60  0000 C CNN
 F 2 "~" H 5900 2500 60  0000 C CNN
@@
 $EndComp
 $Comp
-L 7SEGM S?
+L 7SEGM S5
 U 1 1 53473159
 P 7600 2500
-F 0 "S?" H 7600 3150 60  0000 C CNN
+F 0 "S5" H 7600 3150 60  0000 C CNN
 F 1 "7SEGM" H 7600 1850 60  0000 C CNN
 F 2 "~" H 7600 2500 60  0000 C CNN
@@
 $EndComp
 $Comp
-L 7SEGM S?
+L 7SEGM S6
 U 1 1 5347315F
 P 9250 2500
-F 0 "S?" H 9250 3150 60  0000 C CNN
+F 0 "S6" H 9250 3150 60  0000 C CNN
 F 1 "7SEGM" H 9250 1850 60  0000 C CNN
 F 2 "~" H 9250 2500 60  0000 C CNN
@@
 $EndComp
 Wire Wire Line
-	1800 3750 1750 3750
-Wire Wire Line
-	1750 3750 1750 3950
-Wire Wire Line
-	1750 3950 6850 3950
+	2200 3950 6850 3950
 Wire Wire Line
 	6850 3950 6850 3000
@@
 Connection ~ 3450 3950
 $Comp
-L VCC #PWR?
+L VCC #PWR114
 U 1 1 5347319D
-P 1800 1250
-F 0 "#PWR?" H 1800 1350 30  0001 C CNN
-F 1 "VCC" H 1800 1350 30  0000 C CNN
-F 2 "" H 1800 1250 60  0000 C CNN
-F 3 "" H 1800 1250 60  0000 C CNN
-	1    1800 1250
-	1    0    0    -1
-$EndComp
-$Comp
-L GND #PWR?
+P 2200 1250
+F 0 "#PWR114" H 2200 1350 30  0001 C CNN
+F 1 "VCC" H 2200 1350 30  0000 C CNN
+F 2 "" H 2200 1250 60  0000 C CNN
+F 3 "" H 2200 1250 60  0000 C CNN
+	1    2200 1250
+	0    -1   -1   0
+$EndComp
+$Comp
+L GND #PWR112
 U 1 1 534731B3
 P 1100 2550
-F 0 "#PWR?" H 1100 2550 30  0001 C CNN
+F 0 "#PWR112" H 1100 2550 30  0001 C CNN
 F 1 "GND" H 1100 2480 30  0001 C CNN
 F 2 "" H 1100 2550 60  0000 C CNN
@@
 DISPLAY
 Wire Wire Line
-	8500 2100 8500 1250
-Wire Wire Line
-	8500 1250 2200 1250
+	8500 1250 8500 2100
+Wire Wire Line
+	2600 1250 8500 1250
 Wire Wire Line
 	5150 2100 5150 1250
 Connection ~ 5150 1250
+Text HLabel 1100 2050 0    28   Input ~ 0
+SCL
+Text HLabel 1100 2250 0    28   Input ~ 0
+SDA
+Wire Wire Line
+	2400 1550 2000 1550
+Wire Wire Line
+	2400 3450 2000 3450
+Wire Wire Line
+	2200 3950 2200 3750
 $EndSCHEMATC

Commit message: MLS800  * Fixed missing non connected symbols
Connections:
- no-connect marks 0 -> 4
Changed lines of the file:
@@
 $Descr A4 11693 8268
 encoding utf-8
-Sheet 3 4
+Sheet 2 4
 Title ""
 Date "23 jun 2014"
@@
 $EndComp
 $Comp
-L VCC #PWR111
+L VCC #PWR038
 U 1 1 534730B8
 P 1100 1650
-F 0 "#PWR111" H 1100 1750 30  0001 C CNN
+F 0 "#PWR038" H 1100 1750 30  0001 C CNN
 F 1 "VCC" H 1100 1750 30  0000 C CNN
 F 2 "" H 1100 1650 60  0000 C CNN
@@
 $EndComp
 $Comp
-L GND #PWR113
+L GND #PWR039
 U 1 1 534730C7
 P 1100 3350
-F 0 "#PWR113" H 1100 3350 30  0001 C CNN
+F 0 "#PWR039" H 1100 3350 30  0001 C CNN
 F 1 "GND" H 1100 3280 30  0001 C CNN
 F 2 "" H 1100 3350 60  0000 C CNN
@@
 $EndComp
 $Comp
-L GND #PWR108
+L GND #PWR040
 U 1 1 534730F6
 P 700 2850
-F 0 "#PWR108" H 700 2850 30  0001 C CNN
+F 0 "#PWR040" H 700 2850 30  0001 C CNN
 F 1 "GND" H 700 2780 30  0001 C CNN
 F 2 "" H 700 2850 60  0000 C CNN
@@
 $EndComp
 $Comp
-L GND #PWR110
+L GND #PWR041
 U 1 1 53473118
 P 800 2500
-F 0 "#PWR110" H 800 2500 30  0001 C CNN
+F 0 "#PWR041" H 800 2500 30  0001 C CNN
 F 1 "GND" H 800 2430 30  0001 C CNN
 F 2 "" H 800 2500 60  0000 C CNN
@@
 $EndComp
 $Comp
-L VCC #PWR109
+L VCC #PWR042
 U 1 1 53473123
 P 800 2100
-F 0 "#PWR109" H 800 2200 30  0001 C CNN
+F 0 "#PWR042" H 800 2200 30  0001 C CNN
 F 1 "VCC" H 800 2200 30  0000 C CNN
 F 2 "" H 800 2100 60  0000 C CNN
@@
 $EndComp
 $Comp
-L VCC #PWR115
+L VCC #PWR043
 U 1 1 5347313E
 P 2600 3750
-F 0 "#PWR115" H 2600 3850 30  0001 C CNN
+F 0 "#PWR043" H 2600 3850 30  0001 C CNN
 F 1 "VCC" H 2600 3850 30  0000 C CNN
 F 2 "" H 2600 3750 60  0000 C CNN
@@
 Connection ~ 3450 3950
 $Comp
-L VCC #PWR114
+L VCC #PWR044
 U 1 1 5347319D
 P 2200 1250
-F 0 "#PWR114" H 2200 1350 30  0001 C CNN
+F 0 "#PWR044" H 2200 1350 30  0001 C CNN
 F 1 "VCC" H 2200 1350 30  0000 C CNN
 F 2 "" H 2200 1250 60  0000 C CNN
@@
 $EndComp
 $Comp
-L GND #PWR112
+L GND #PWR045
 U 1 1 534731B3
 P 1100 2550
-F 0 "#PWR112" H 1100 2550 30  0001 C CNN
+F 0 "#PWR045" H 1100 2550 30  0001 C CNN
 F 1 "GND" H 1100 2480 30  0001 C CNN
 F 2 "" H 1100 2550 60  0000 C CNN
@@
 Wire Wire Line
 	2000 3150 2100 3150
-Wire Wire Line
-	2000 3250 2100 3250
 Entry Wire Line
 	2100 1750 2200 1850
@@
 	6750 2100 6850 2200
 Entry Wire Line
-	6750 2000 6850 2100
-Entry Wire Line
 	8400 2700 8500 2800
 Entry Wire Line
@@
 Wire Wire Line
 	2200 3950 2200 3750
+Wire Wire Line
+	2000 3250 2100 3250
+NoConn ~ 5150 3000
+NoConn ~ 3450 2100
+NoConn ~ 6850 2100
+NoConn ~ 8500 3000
+Text Label 3450 2200 0    28   ~ 0
+1a
+Text Label 3450 2300 0    28   ~ 0
+1b
+Text Label 3450 2400 0    28   ~ 0
+1c
+Text Label 3450 2500 0    28   ~ 0
+1d
+Text Label 3450 2600 0    28   ~ 0
+1e
+Text Label 3450 2700 0    28   ~ 0
+1f
+Text Label 3450 2800 0    28   ~ 0
+1g
+Text Label 3450 2900 0    28   ~ 0
+1dp
+Text Label 5150 2900 0    28   ~ 0
+1dp
+Text Label 5150 2800 0    28   ~ 0
+1g
+Entry Wire Line
+	5050 2600 5150 2700
+Text Label 5150 2700 0    28   ~ 0
+1f
+Text Label 5150 2600 0    28   ~ 0
+1e
+Text Label 5150 2500 0    28   ~ 0
+1d
+Text Label 5150 2400 0    28   ~ 0
+1c
+Text Label 5150 2300 0    28   ~ 0
+1b
+Text Label 5150 2200 0    28   ~ 0
+1a
+Text Label 6850 2200 0    28   ~ 0
+2a
+Text Label 6850 2300 0    28   ~ 0
+2b
+Text Label 6850 2400 0    28   ~ 0
+2c
+Text Label 6850 2500 0    28   ~ 0
+2d
+Text Label 6850 2600 0    28   ~ 0
+2e
+Text Label 6850 2700 0    28   ~ 0
+2f
+Text Label 6850 2800 0    28   ~ 0
+2g
+Text Label 6850 2900 0    28   ~ 0
+2dp
+Text Label 8500 2200 0    28   ~ 0
+2a
+Text Label 8500 2300 0    28   ~ 0
+2b
+Text Label 8500 2400 0    28   ~ 0
+2c
+Text Label 8500 2500 0    28   ~ 0
+2d
+Text Label 8500 2600 0    28   ~ 0
+2e
+Text Label 8500 2700 0    28   ~ 0
+2f
+Text Label 8500 2800 0    28   ~ 0
+2g
+Text Label 8500 2900 0    28   ~ 0
+2dp
 $EndSCHEMATC

Commit message: MLS800  * Fixed some crc errors  * Fixed wrong AREF/UCAP schematics  * Generated netlist
Parts:
- renumbered C11 to C12, C12 to C13, Q17 to Q1, Q18 to Q2
Changed lines of the file:
@@
 Sheet 2 4
 Title ""
-Date "23 jun 2014"
+Date "24 jun 2014"
 Rev ""
 Comp ""
@@
 $EndComp
 $Comp
-L VCC #PWR038
+L VCC #PWR036
 U 1 1 534730B8
 P 1100 1650
-F 0 "#PWR038" H 1100 1750 30  0001 C CNN
+F 0 "#PWR036" H 1100 1750 30  0001 C CNN
 F 1 "VCC" H 1100 1750 30  0000 C CNN
 F 2 "" H 1100 1650 60  0000 C CNN
@@
 $EndComp
 $Comp
-L GND #PWR039
+L GND #PWR037
 U 1 1 534730C7
 P 1100 3350
-F 0 "#PWR039" H 1100 3350 30  0001 C CNN
+F 0 "#PWR037" H 1100 3350 30  0001 C CNN
 F 1 "GND" H 1100 3280 30  0001 C CNN
 F 2 "" H 1100 3350 60  0000 C CNN
@@
 $EndComp
 $Comp
-L C C12
+L C C13
 U 1 1 534730D6
 P 900 2850
-F 0 "C12" H 900 2950 40  0000 L CNN
+F 0 "C13" H 900 2950 40  0000 L CNN
 F 1 "2.7nF" H 906 2765 40  0000 L CNN
 F 2 "~" H 938 2700 30  0000 C CNN
@@
 $EndComp
 $Comp
-L GND #PWR040
+L GND #PWR038
 U 1 1 534730F6
 P 700 2850
-F 0 "#PWR040" H 700 2850 30  0001 C CNN
+F 0 "#PWR038" H 700 2850 30  0001 C CNN
 F 1 "GND" H 700 2780 30  0001 C CNN
 F 2 "" H 700 2850 60  0000 C CNN
@@
 $EndComp
 $Comp
-L C C11
+L C C12
 U 1 1 534730FC
 P 800 2300
-F 0 "C11" H 800 2400 40  0000 L CNN
+F 0 "C12" H 800 2400 40  0000 L CNN
 F 1 "100nF" H 806 2215 40  0000 L CNN
 F 2 "~" H 838 2150 30  0000 C CNN
@@
 $EndComp
 $Comp
-L GND #PWR041
+L GND #PWR039
 U 1 1 53473118
 P 800 2500
-F 0 "#PWR041" H 800 2500 30  0001 C CNN
+F 0 "#PWR039" H 800 2500 30  0001 C CNN
 F 1 "GND" H 800 2430 30  0001 C CNN
 F 2 "" H 800 2500 60  0000 C CNN
@@
 $EndComp
 $Comp
-L VCC #PWR042
+L VCC #PWR040
 U 1 1 53473123
 P 800 2100
-F 0 "#PWR042" H 800 2200 30  0001 C CNN
+F 0 "#PWR040" H 800 2200 30  0001 C CNN
 F 1 "VCC" H 800 2200 30  0000 C CNN
 F 2 "" H 800 2100 60  0000 C CNN
@@
 $EndComp
 $Comp
-L NPN Q18
+L NPN Q2
 U 1 1 5347312B
 P 2400 3650
-F 0 "Q18" H 2400 3500 50  0000 R CNN
+F 0 "Q2" H 2400 3500 50  0000 R CNN
 F 1 "NPN" H 2400 3800 50  0000 R CNN
 F 2 "~" H 2400 3650 60  0000 C CNN
@@
 $EndComp
 $Comp
-L NPN Q17
+L NPN Q1
 U 1 1 53473138
 P 2400 1350
-F 0 "Q17" H 2400 1200 50  0000 R CNN
+F 0 "Q1" H 2400 1200 50  0000 R CNN
 F 1 "NPN" H 2400 1500 50  0000 R CNN
 F 2 "~" H 2400 1350 60  0000 C CNN
@@
 $EndComp
 $Comp
-L VCC #PWR043
+L VCC #PWR041
 U 1 1 5347313E
 P 2600 3750
-F 0 "#PWR043" H 2600 3850 30  0001 C CNN
+F 0 "#PWR041" H 2600 3850 30  0001 C CNN
 F 1 "VCC" H 2600 3850 30  0000 C CNN
 F 2 "" H 2600 3750 60  0000 C CNN
@@
 Connection ~ 3450 3950
 $Comp
-L VCC #PWR044
+L VCC #PWR042
 U 1 1 5347319D
 P 2200 1250
-F 0 "#PWR044" H 2200 1350 30  0001 C CNN
+F 0 "#PWR042" H 2200 1350 30  0001 C CNN
 F 1 "VCC" H 2200 1350 30  0000 C CNN
 F 2 "" H 2200 1250 60  0000 C CNN
@@
 $EndComp
 $Comp
-L GND #PWR045
+L GND #PWR043
 U 1 1 534731B3
 P 1100 2550
-F 0 "#PWR045" H 1100 2550 30  0001 C CNN
+F 0 "#PWR043" H 1100 2550 30  0001 C CNN
 F 1 "GND" H 1100 2480 30  0001 C CNN
 F 2 "" H 1100 2550 60  0000 C CNN

Commit message: MLS800  * Added separated GND : AGND & GND  * Revamped the loops schema  * Put values on all components  * Started to add footprint annotations to some resistors
Parts:
- Q1, Q2: value NPN -> 2N3904
Connections:
- net labels added: DGND
- net labels removed: GND
- wire segments 25 -> 47
- no-connect marks 4 -> 0
Other:
- moved on the sheet: C12, C13, IC2, Q1, Q2

Commit message: MLS800  * Started cmp association
Parts:
- removed S3, S4, S5, S6: 7SEGM, ~, symbol 7SEGM
- added S1, S2: 7SEGM_DBL, ~, symbol 7SEGM_DBL
Connections:
- wire segments 47 -> 33
Changed lines of the file:
@@
 Sheet 2 4
 Title ""
-Date "17 aug 2014"
+Date "18 aug 2014"
 Rev ""
 Comp ""
@@
 $EndComp
 $Comp
-L VCC #PWR039
+L VCC #PWR37
 U 1 1 534730B8
 P 700 1650
-F 0 "#PWR039" H 700 1750 30  0001 C CNN
+F 0 "#PWR37" H 700 1750 30  0001 C CNN
 F 1 "VCC" H 700 1750 30  0000 C CNN
 F 2 "" H 700 1650 60  0000 C CNN
@@
 $EndComp
 $Comp
-L VCC #PWR040
+L VCC #PWR42
 U 1 1 5347313E
 P 2850 3750
-F 0 "#PWR040" H 2850 3850 30  0001 C CNN
+F 0 "#PWR42" H 2850 3850 30  0001 C CNN
 F 1 "VCC" H 2850 3850 30  0000 C CNN
 F 2 "" H 2850 3750 60  0000 C CNN
@@
 $EndComp
 $Comp
-L 7SEGM S3
-U 1 1 53473146
-P 4450 2500
-F 0 "S3" H 4450 3150 60  0000 C CNN
-F 1 "7SEGM" H 4450 1850 60  0000 C CNN
-F 2 "~" H 4450 2500 60  0000 C CNN
-F 3 "~" H 4450 2500 60  0000 C CNN
-	1    4450 2500
-	1    0    0    -1
-$EndComp
-$Comp
-L 7SEGM S4
-U 1 1 53473153
-P 6150 2500
-F 0 "S4" H 6150 3150 60  0000 C CNN
-F 1 "7SEGM" H 6150 1850 60  0000 C CNN
-F 2 "~" H 6150 2500 60  0000 C CNN
-F 3 "~" H 6150 2500 60  0000 C CNN
-	1    6150 2500
-	1    0    0    -1
-$EndComp
-$Comp
-L 7SEGM S5
-U 1 1 53473159
-P 7850 2500
-F 0 "S5" H 7850 3150 60  0000 C CNN
-F 1 "7SEGM" H 7850 1850 60  0000 C CNN
-F 2 "~" H 7850 2500 60  0000 C CNN
-F 3 "~" H 7850 2500 60  0000 C CNN
-	1    7850 2500
-	1    0    0    -1
-$EndComp
-$Comp
-L 7SEGM S6
-U 1 1 5347315F
-P 9500 2500
-F 0 "S6" H 9500 3150 60  0000 C CNN
-F 1 "7SEGM" H 9500 1850 60  0000 C CNN
-F 2 "~" H 9500 2500 60  0000 C CNN
-F 3 "~" H 9500 2500 60  0000 C CNN
-	1    9500 2500
-	1    0    0    -1
-$EndComp
-Wire Wire Line
-	2450 3950 7100 3950
-Wire Wire Line
-	7100 3950 7100 3000
-Wire Wire Line
-	3700 3000 3700 3950
-Connection ~ 3700 3950
-$Comp
-L VCC #PWR041
+L VCC #PWR41
 U 1 1 5347319D
 P 2450 1250
-F 0 "#PWR041" H 2450 1350 30  0001 C CNN
+F 0 "#PWR41" H 2450 1350 30  0001 C CNN
 F 1 "VCC" H 2450 1350 30  0000 C CNN
 F 2 "" H 2450 1250 60  0000 C CNN
@@
 DISPLAY
 Wire Wire Line
-	8750 1250 8750 2100
-Wire Wire Line
 	2850 1250 8750 1250
-Wire Wire Line
-	5400 2100 5400 1250
-Connection ~ 5400 1250
 Text HLabel 1350 2050 0    28   Input ~ 0
 SCL
@@
 2dp
 $Comp
-L DGND #PWR042
+L DGND #PWR38
 U 1 1 53F19FF1
 P 700 3450
-F 0 "#PWR042" H 700 3450 40  0001 C CNN
+F 0 "#PWR38" H 700 3450 40  0001 C CNN
 F 1 "DGND" H 700 3380 40  0000 C CNN
 F 2 "" H 700 3450 60  0000 C CNN
@@
 $EndComp
 $Comp
-L DGND #PWR043
+L DGND #PWR39
 U 1 1 53F19FFE
 P 950 2850
-F 0 "#PWR043" H 950 2850 40  0001 C CNN
+F 0 "#PWR39" H 950 2850 40  0001 C CNN
 F 1 "DGND" H 950 2780 40  0000 C CNN
 F 2 "" H 950 2850 60  0000 C CNN
@@
 $EndComp
 $Comp
-L DGND #PWR044
+L DGND #PWR40
 U 1 1 53F1A004
 P 1350 2550
-F 0 "#PWR044" H 1350 2550 40  0001 C CNN
+F 0 "#PWR40" H 1350 2550 40  0001 C CNN
 F 1 "DGND" H 1350 2480 40  0000 C CNN
 F 2 "" H 1350 2550 60  0000 C CNN
@@
 Connection ~ 700  3350
 Wire Wire Line
-	3700 3000 3500 3000
-Wire Wire Line
-	3500 3000 3500 2050
+	3500 2050 3500 3950
 Wire Wire Line
 	3500 2050 3700 2050
@@
 	3700 2050 3700 2100
 Wire Wire Line
-	5400 2100 5350 2100
-Wire Wire Line
-	5350 2100 5350 2050
-Wire Wire Line
-	5400 3000 5200 3000
-Wire Wire Line
-	5200 3000 5200 2050
-Wire Wire Line
-	5200 2050 5350 2050
-Wire Wire Line
-	7100 3000 6900 3000
-Wire Wire Line
-	6900 3000 6900 2050
+	6900 3950 6900 2050
 Wire Wire Line
 	6900 2050 7100 2050
 Wire Wire Line
 	7100 2050 7100 2100
-Wire Wire Line
-	8750 3000 8550 3000
-Wire Wire Line
-	8550 3000 8550 2050
-Wire Wire Line
-	8550 2050 8700 2050
-Wire Wire Line
-	8700 2050 8700 2100
-Wire Wire Line
-	8700 2100 8750 2100
+$Comp
+L 7SEGM_DBL S1
+U 1 1 53F13A39
+P 4450 2500
+F 0 "S1" H 4450 3150 60  0000 C CNN
+F 1 "7SEGM_DBL" H 4450 1850 60  0000 C CNN
+F 2 "~" H 4450 2500 60  0000 C CNN
+F 3 "~" H 4450 2500 60  0000 C CNN
+	1    4450 2500
+	1    0    0    -1
+$EndComp
+$Comp
+L 7SEGM_DBL S1
+U 2 1 53F13A46
+P 6150 2500
+F 0 "S1" H 6150 3150 60  0000 C CNN
+F 1 "7SEGM_DBL" H 6150 1850 60  0000 C CNN
+F 2 "~" H 6150 2500 60  0000 C CNN
+F 3 "~" H 6150 2500 60  0000 C CNN
+	2    6150 2500
+	1    0    0    -1
+$EndComp
+$Comp
+L 7SEGM_DBL S2
+U 1 1 53F13A4C
+P 7850 2500
+F 0 "S2" H 7850 3150 60  0000 C CNN
+F 1 "7SEGM_DBL" H 7850 1850 60  0000 C CNN
+F 2 "~" H 7850 2500 60  0000 C CNN
+F 3 "~" H 7850 2500 60  0000 C CNN
+	1    7850 2500
+	1    0    0    -1
+$EndComp
+$Comp
+L 7SEGM_DBL S2
+U 2 1 53F13A52
+P 9500 2500
+F 0 "S2" H 9500 3150 60  0000 C CNN
+F 1 "7SEGM_DBL" H 9500 1850 60  0000 C CNN
+F 2 "~" H 9500 2500 60  0000 C CNN
+F 3 "~" H 9500 2500 60  0000 C CNN
+	2    9500 2500
+	1    0    0    -1
+$EndComp
+Wire Wire Line
+	8750 1250 8750 2100
+Wire Wire Line
+	2450 3950 6900 3950
+Connection ~ 3500 3950
+Wire Wire Line
+	5400 2100 5400 1250
+Connection ~ 5400 1250
 $EndSCHEMATC

Commit message: MLS800 :  - assigning footprints
Parts:
- C13: renamed from C12; footprint ~ -> Capacitors_SMD:c_0805
- C14: renamed from C13; footprint ~ -> Capacitors_SMD:c_0805
Changed lines of the file:
@@
 $EndComp
 $Comp
-L C C13
+L C C14
 U 1 1 534730D6
 P 1150 2850
-F 0 "C13" H 1150 2950 40  0000 L CNN
+F 0 "C14" H 1150 2950 40  0000 L CNN
 F 1 "2.7nF" H 1156 2765 40  0000 L CNN
-F 2 "~" H 1188 2700 30  0000 C CNN
+F 2 "Capacitors_SMD:c_0805" H 1188 2700 30  0001 C CNN
 F 3 "~" H 1150 2850 60  0000 C CNN
 	1    1150 2850
@@
 $EndComp
 $Comp
-L C C12
+L C C13
 U 1 1 534730FC
 P 700 2300
-F 0 "C12" H 700 2400 40  0000 L CNN
+F 0 "C13" H 700 2400 40  0000 L CNN
 F 1 "100nF" H 706 2215 40  0000 L CNN
-F 2 "~" H 738 2150 30  0000 C CNN
+F 2 "Capacitors_SMD:c_0805" H 738 2150 30  0001 C CNN
 F 3 "~" H 700 2300 60  0000 C CNN
 	1    700  2300
