File: mls800_display.sch (KiCad schematic (older format))
At the start: 7 parts, among them IC2 SAA1064T, Q1 2N3904, Q2 2N3904

Commit message: MLS800 : disabled switch tact led "interchangeable" units => fixed annotations
MLS800 : front panel schematic seems to be completed
Parts:
- renumbered S1 to S?, S2 to S?
Changed lines of the file:
@@
 $EndComp
 $Comp
-L VCC #PWR039
+L VCC #PWR37
 U 1 1 534730B8
 P 700 1650
-F 0 "#PWR039" H 700 1750 30  0001 C CNN
+F 0 "#PWR37" H 700 1750 30  0001 C CNN
 F 1 "VCC" H 700 1750 30  0000 C CNN
 F 2 "" H 700 1650 60  0000 C CNN
@@
 $EndComp
 $Comp
-L VCC #PWR040
+L VCC #PWR42
 U 1 1 5347313E
 P 2850 3750
-F 0 "#PWR040" H 2850 3850 30  0001 C CNN
+F 0 "#PWR42" H 2850 3850 30  0001 C CNN
 F 1 "VCC" H 2850 3850 30  0000 C CNN
 F 2 "" H 2850 3750 60  0000 C CNN
@@
 $EndComp
 $Comp
-L VCC #PWR041
+L VCC #PWR41
 U 1 1 5347319D
 P 2450 1250
-F 0 "#PWR041" H 2450 1350 30  0001 C CNN
+F 0 "#PWR41" H 2450 1350 30  0001 C CNN
 F 1 "VCC" H 2450 1350 30  0000 C CNN
 F 2 "" H 2450 1250 60  0000 C CNN
@@
 2dp
 $Comp
-L DGND #PWR042
+L DGND #PWR38
 U 1 1 53F19FF1
 P 700 3450
-F 0 "#PWR042" H 700 3450 40  0001 C CNN
+F 0 "#PWR38" H 700 3450 40  0001 C CNN
 F 1 "DGND" H 700 3380 40  0000 C CNN
 F 2 "" H 700 3450 60  0000 C CNN
@@
 $EndComp
 $Comp
-L DGND #PWR043
+L DGND #PWR39
 U 1 1 53F19FFE
 P 950 2850
-F 0 "#PWR043" H 950 2850 40  0001 C CNN
+F 0 "#PWR39" H 950 2850 40  0001 C CNN
 F 1 "DGND" H 950 2780 40  0000 C CNN
 F 2 "" H 950 2850 60  0000 C CNN
@@
 $EndComp
 $Comp
-L DGND #PWR044
+L DGND #PWR40
 U 1 1 53F1A004
 P 1350 2550
-F 0 "#PWR044" H 1350 2550 40  0001 C CNN
+F 0 "#PWR40" H 1350 2550 40  0001 C CNN
 F 1 "DGND" H 1350 2480 40  0000 C CNN
 F 2 "" H 1350 2550 60  0000 C CNN
@@
 	7100 2050 7100 2100
 $Comp
-L 7SEGM_DBL S1
+L 7SEGM_DBL S?
 U 1 1 53F13A39
 P 4450 2500
-F 0 "S1" H 4450 3150 60  0000 C CNN
+F 0 "S?" H 4450 3150 60  0000 C CNN
 F 1 "7SEGM_DBL" H 4450 1850 60  0000 C CNN
 F 2 "~" H 4450 2500 60  0000 C CNN
@@
 $EndComp
 $Comp
-L 7SEGM_DBL S1
-U 2 1 53F13A46
+L 7SEGM_DBL S?
+U 1 1 53F13A46
 P 6150 2500
-F 0 "S1" H 6150 3150 60  0000 C CNN
+F 0 "S?" H 6150 3150 60  0000 C CNN
 F 1 "7SEGM_DBL" H 6150 1850 60  0000 C CNN
 F 2 "~" H 6150 2500 60  0000 C CNN
 F 3 "~" H 6150 2500 60  0000 C CNN
-	2    6150 2500
-	1    0    0    -1
-$EndComp
-$Comp
-L 7SEGM_DBL S2
+	1    6150 2500
+	1    0    0    -1
+$EndComp
+$Comp
+L 7SEGM_DBL S?
 U 1 1 53F13A4C
 P 7850 2500
-F 0 "S2" H 7850 3150 60  0000 C CNN
+F 0 "S?" H 7850 3150 60  0000 C CNN
 F 1 "7SEGM_DBL" H 7850 1850 60  0000 C CNN
 F 2 "~" H 7850 2500 60  0000 C CNN
@@
 $EndComp
 $Comp
-L 7SEGM_DBL S2
-U 2 1 53F13A52
+L 7SEGM_DBL S?
+U 1 1 53F13A52
 P 9500 2500
-F 0 "S2" H 9500 3150 60  0000 C CNN
+F 0 "S?" H 9500 3150 60  0000 C CNN
 F 1 "7SEGM_DBL" H 9500 1850 60  0000 C CNN
 F 2 "~" H 9500 2500 60  0000 C CNN
 F 3 "~" H 9500 2500 60  0000 C CNN
-	2    9500 2500
-	1    0    0    -1
-$EndComp
+	1    9500 2500
+	1    0    0    -1
+$EndComp
