File: mls800_misc.sch (KiCad schematic (older format))
At the start: 26 parts

Commit message: MLS800  * Lots of change in diagram/schematic  * Added external parts
Parts:
- removed D?: DIODE, ~, symbol DIODE
- removed IC?: 6N137, DIP8, symbol 6N137
- removed P? (x2): DIN_5, symbol DIN_5
- removed R? (x3): 220R, ~, symbol R
- removed U?: 24LC256, symbol 24LC256
- gave numbers to parts that had none: 18
Connections:
- net labels removed: RX
- wire segments 95 -> 77
Other:
- note removed: "MEM\n"
- note removed: "MIDI\n"

Commit message: MLS800  * Fixed missing non connected symbols
Connections:
- net labels removed: l8
- no-connect marks 0 -> 1
Changed lines of the file:
@@
 $Descr A4 11693 8268
 encoding utf-8
-Sheet 4 4
+Sheet 3 4
 Title ""
 Date "23 jun 2014"
@@
 $EndComp
 $Comp
-L VCC #PWR118
+L VCC #PWR046
 U 1 1 5350562C
 P 2150 1100
-F 0 "#PWR118" H 2150 1200 30  0001 C CNN
+F 0 "#PWR046" H 2150 1200 30  0001 C CNN
 F 1 "VCC" H 2150 1200 30  0000 C CNN
 F 2 "" H 2150 1100 60  0000 C CNN
@@
 $EndComp
 $Comp
-L GND #PWR119
+L GND #PWR047
 U 1 1 53505632
 P 2150 3800
-F 0 "#PWR119" H 2150 3800 30  0001 C CNN
+F 0 "#PWR047" H 2150 3800 30  0001 C CNN
 F 1 "GND" H 2150 3730 30  0001 C CNN
 F 2 "" H 2150 3800 60  0000 C CNN
@@
 $EndComp
 $Comp
-L GND #PWR117
+L GND #PWR048
 U 1 1 5350563A
 P 1100 2100
-F 0 "#PWR117" H 1100 2100 30  0001 C CNN
+F 0 "#PWR048" H 1100 2100 30  0001 C CNN
 F 1 "GND" H 1100 2030 30  0001 C CNN
 F 2 "" H 1100 2100 60  0000 C CNN
@@
 $EndComp
 $Comp
-L GND #PWR116
+L GND #PWR049
 U 1 1 53505646
 P 700 1550
-F 0 "#PWR116" H 700 1550 30  0001 C CNN
+F 0 "#PWR049" H 700 1550 30  0001 C CNN
 F 1 "GND" H 700 1480 30  0001 C CNN
 F 2 "" H 700 1550 60  0000 C CNN
@@
 Entry Wire Line
 	3200 2150 3300 2250
-Entry Wire Line
-	3200 2250 3300 2350
 Text Label 4450 1300 0    60   ~ 0
 I1
@@
 	3550 4300 3650 4400
 Text Label 4450 5150 0    60   ~ 0
-l8
+I8
 $Comp
 L SW_TACT_LED S14
@@
 Entry Wire Line
 	4350 5050 4450 5150
-Entry Wire Line
-	3550 4850 3650 4950
-Connection ~ 1150 2100
-Wire Wire Line
-	1100 2100 1200 2100
-Wire Wire Line
-	1150 2200 1200 2200
-Wire Wire Line
-	1150 2000 1150 2200
-Wire Wire Line
-	1200 2000 1150 2000
-Wire Wire Line
-	3100 3100 3200 3100
-Wire Wire Line
-	3100 3000 3200 3000
-Wire Wire Line
-	3100 2900 3200 2900
-Wire Wire Line
-	3100 2800 3200 2800
-Wire Wire Line
-	3100 2700 3200 2700
-Wire Wire Line
-	3100 2600 3200 2600
-Wire Wire Line
-	3100 2500 3200 2500
-Wire Wire Line
-	3100 2400 3200 2400
-Wire Wire Line
-	3100 1550 3200 1550
-Wire Wire Line
-	3100 1650 3200 1650
-Wire Wire Line
-	3100 1750 3200 1750
-Wire Wire Line
-	3100 1850 3200 1850
-Wire Wire Line
-	3100 1950 3200 1950
-Wire Wire Line
-	3100 2050 3200 2050
-Wire Wire Line
-	3100 2150 3200 2150
-Wire Wire Line
-	3100 2250 3200 2250
-Wire Wire Line
-	4550 1300 4550 1200
-Wire Wire Line
-	4550 1850 4550 1750
-Wire Wire Line
-	4550 2400 4550 2300
-Wire Wire Line
-	4550 2950 4550 2850
-Wire Wire Line
-	4550 3500 4550 3400
-Wire Wire Line
-	4550 4050 4550 3950
-Wire Wire Line
-	4550 4600 4550 4500
-Wire Wire Line
-	4550 5150 4550 5050
-Wire Bus Line
-	3300 900  3300 2350
-Wire Wire Line
-	5050 1100 5150 1100
-Wire Wire Line
-	5150 1100 5150 5150
-Wire Wire Line
-	5050 5150 5250 5150
-Wire Wire Line
-	5050 5050 5150 5050
-Connection ~ 5150 5050
-Wire Wire Line
-	5050 4950 5150 4950
-Connection ~ 5150 4950
-Wire Wire Line
-	5050 4600 5150 4600
-Connection ~ 5150 4600
-Wire Wire Line
-	5050 4500 5150 4500
-Connection ~ 5150 4500
-Wire Wire Line
-	5050 4400 5150 4400
-Connection ~ 5150 4400
-Wire Wire Line
-	5050 4050 5150 4050
-Connection ~ 5150 4050
-Wire Wire Line
-	5050 3950 5150 3950
-Connection ~ 5150 3950
-Wire Wire Line
-	5050 3850 5150 3850
-Connection ~ 5150 3850
-Wire Wire Line
-	5050 3500 5150 3500
-Connection ~ 5150 3500
-Wire Wire Line
-	5050 3400 5150 3400
-Connection ~ 5150 3400
-Wire Wire Line
-	5050 3300 5150 3300
-Connection ~ 5150 3300
-Wire Wire Line
-	5050 2950 5150 2950
-Connection ~ 5150 2950
-Wire Wire Line
-	5050 2850 5150 2850
-Connection ~ 5150 2850
-Wire Wire Line
-	5050 2750 5150 2750
-Connection ~ 5150 2750
-Wire Wire Line
-	5050 2400 5150 2400
-Connection ~ 5150 2400
-Wire Wire Line
-	5050 2300 5150 2300
-Connection ~ 5150 2300
-Wire Wire Line
-	5050 2200 5150 2200
-Connection ~ 5150 2200
-Wire Wire Line
-	5050 1850 5150 1850
-Connection ~ 5150 1850
-Wire Wire Line
-	5050 1750 5150 1750
-Connection ~ 5150 1750
-Wire Wire Line
-	5050 1650 5150 1650
-Connection ~ 5150 1650
-Wire Wire Line
-	5050 1200 5150 1200
-Connection ~ 5150 1200
-Wire Wire Line
-	5050 1300 5150 1300
-Connection ~ 5150 1300
-$Comp
-L GND #PWR120
+$Comp
+L GND #PWR050
 U 1 1 537951D0
 P 5250 5150
-F 0 "#PWR120" H 5250 5150 30  0001 C CNN
+F 0 "#PWR050" H 5250 5150 30  0001 C CNN
 F 1 "GND" H 5250 5080 30  0001 C CNN
 F 2 "" H 5250 5150 60  0000 C CNN
@@
 	0    -1   -1   0
 $EndComp
-Connection ~ 5150 5150
 Text Label 3650 1100 0    60   ~ 0
 L1
-Wire Wire Line
-	3650 4950 3750 4950
-Wire Wire Line
-	3650 4400 3750 4400
-Wire Wire Line
-	3650 3850 3750 3850
-Wire Wire Line
-	3650 3300 3750 3300
-Wire Wire Line
-	3650 2750 3750 2750
-Wire Wire Line
-	3650 2200 3750 2200
-Wire Wire Line
-	3650 1650 3750 1650
-Wire Wire Line
-	3650 1100 3750 1100
 Text Label 3650 1650 0    60   ~ 0
 L2
@@
 Text Label 3650 4400 0    60   ~ 0
 L7
-Text Label 3650 4950 0    60   ~ 0
-L8
+Text HLabel 1200 2950 0    28   Input ~ 0
+SDA
+Text HLabel 1200 3050 0    28   Input ~ 0
+SCL
+Text HLabel 3100 3350 2    28   Input ~ 0
+UI INT
+NoConn ~ 3100 3250
+Entry Wire Line
+	3200 2250 3300 2350
+Connection ~ 1150 2100
+Wire Wire Line
+	1100 2100 1200 2100
+Wire Wire Line
+	1150 2200 1200 2200
+Wire Wire Line
+	1150 2000 1150 2200
+Wire Wire Line
+	1200 2000 1150 2000
+Wire Wire Line
+	3100 3100 3200 3100
+Wire Wire Line
+	3100 3000 3200 3000
+Wire Wire Line
+	3100 2900 3200 2900
+Wire Wire Line
+	3100 2800 3200 2800
+Wire Wire Line
+	3100 2700 3200 2700
+Wire Wire Line
+	3100 2600 3200 2600
+Wire Wire Line
+	3100 2500 3200 2500
+Wire Wire Line
+	3100 2400 3200 2400
+Wire Wire Line
+	3100 1550 3200 1550
+Wire Wire Line
+	3100 1650 3200 1650
+Wire Wire Line
+	3100 1750 3200 1750
+Wire Wire Line
+	3100 1850 3200 1850
+Wire Wire Line
+	3100 1950 3200 1950
+Wire Wire Line
+	3100 2050 3200 2050
+Wire Wire Line
+	3100 2150 3200 2150
+Wire Wire Line
+	4550 1300 4550 1200
+Wire Wire Line
+	4550 1850 4550 1750
+Wire Wire Line
+	4550 2400 4550 2300
+Wire Wire Line
+	4550 2950 4550 2850
+Wire Wire Line
+	4550 3500 4550 3400
+Wire Wire Line
+	4550 4050 4550 3950
+Wire Wire Line
+	4550 4600 4550 4500
+Wire Wire Line
+	4550 5150 4550 5050
+Wire Bus Line
+	3300 900  3300 2350
+Wire Wire Line
+	5050 1100 5150 1100
+Wire Wire Line
+	5150 1100 5150 5150
+Wire Wire Line
+	5050 5150 5250 5150
+Wire Wire Line
+	5050 5050 5150 5050
+Connection ~ 5150 5050
+Wire Wire Line
+	5050 4950 5150 4950
+Connection ~ 5150 4950
+Wire Wire Line
+	5050 4600 5150 4600
+Connection ~ 5150 4600
+Wire Wire Line
+	5050 4500 5150 4500
+Connection ~ 5150 4500
+Wire Wire Line
+	5050 4400 5150 4400
+Connection ~ 5150 4400
+Wire Wire Line
+	5050 4050 5150 4050
+Connection ~ 5150 4050
+Wire Wire Line
+	5050 3950 5150 3950
+Connection ~ 5150 3950
+Wire Wire Line
+	5050 3850 5150 3850
+Connection ~ 5150 3850
+Wire Wire Line
+	5050 3500 5150 3500
+Connection ~ 5150 3500
+Wire Wire Line
+	5050 3400 5150 3400
+Connection ~ 5150 3400
+Wire Wire Line
+	5050 3300 5150 3300
+Connection ~ 5150 3300
+Wire Wire Line
+	5050 2950 5150 2950
+Connection ~ 5150 2950
+Wire Wire Line
+	5050 2850 5150 2850
+Connection ~ 5150 2850
+Wire Wire Line
+	5050 2750 5150 2750
+Connection ~ 5150 2750
+Wire Wire Line
+	5050 2400 5150 2400
+Connection ~ 5150 2400
+Wire Wire Line
+	5050 2300 5150 2300
+Connection ~ 5150 2300
+Wire Wire Line
+	5050 2200 5150 2200
+Connection ~ 5150 2200
+Wire Wire Line
+	5050 1850 5150 1850
+Connection ~ 5150 1850
+Wire Wire Line
+	5050 1750 5150 1750
+Connection ~ 5150 1750
+Wire Wire Line
+	5050 1650 5150 1650
+Connection ~ 5150 1650
+Wire Wire Line
+	5050 1200 5150 1200
+Connection ~ 5150 1200
+Wire Wire Line
+	5050 1300 5150 1300
+Connection ~ 5150 1300
+Connection ~ 5150 5150
+Wire Wire Line
+	3650 4400 3750 4400
+Wire Wire Line
+	3650 3850 3750 3850
+Wire Wire Line
+	3650 3300 3750 3300
+Wire Wire Line
+	3650 2750 3750 2750
+Wire Wire Line
+	3650 2200 3750 2200
+Wire Wire Line
+	3650 1650 3750 1650
+Wire Wire Line
+	3650 1100 3750 1100
 Wire Bus Line
 	3550 4850 3550 1000
@@
 Wire Bus Line
 	4350 900  4350 5050
-Text HLabel 1200 2950 0    28   Input ~ 0
-SDA
-Text HLabel 1200 3050 0    28   Input ~ 0
-SCL
-Text HLabel 3100 3350 2    28   Input ~ 0
-UI INT
+Wire Wire Line
+	3100 2250 3200 2250
+Text Label 3650 4950 0    60   ~ 0
+L8
+Wire Wire Line
+	3750 4950 3650 4950
+Entry Wire Line
+	3550 4850 3650 4950
 $EndSCHEMATC

Commit message: MLS800  * Fixed some crc errors  * Fixed wrong AREF/UCAP schematics  * Generated netlist
Parts:
- renumbered R16 to R15, R17 to R16, R18 to R17, R19 to R18, R20 to R19, R21 to R20, R22 to R21, R23 to R22, R24 to R23, U5 to U4
Changed lines of the file:
@@
 Sheet 3 4
 Title ""
-Date "23 jun 2014"
+Date "24 jun 2014"
 Rev ""
 Comp ""
@@
 $EndDescr
 $Comp
-L MCP23017 U5
+L MCP23017 U4
 U 1 1 53505620
 P 2150 2450
-F 0 "U5" H 1600 3550 50  0000 C CNN
+F 0 "U4" H 1600 3550 50  0000 C CNN
 F 1 "MCP23017" H 2600 1350 50  0000 C CNN
 F 2 "MODULE" H 1650 1350 50  0001 C CNN
@@
 $EndComp
 $Comp
-L VCC #PWR046
+L VCC #PWR044
 U 1 1 5350562C
 P 2150 1100
-F 0 "#PWR046" H 2150 1200 30  0001 C CNN
+F 0 "#PWR044" H 2150 1200 30  0001 C CNN
 F 1 "VCC" H 2150 1200 30  0000 C CNN
 F 2 "" H 2150 1100 60  0000 C CNN
@@
 $EndComp
 $Comp
-L GND #PWR047
+L GND #PWR045
 U 1 1 53505632
 P 2150 3800
-F 0 "#PWR047" H 2150 3800 30  0001 C CNN
+F 0 "#PWR045" H 2150 3800 30  0001 C CNN
 F 1 "GND" H 2150 3730 30  0001 C CNN
 F 2 "" H 2150 3800 60  0000 C CNN
@@
 $EndComp
 $Comp
-L GND #PWR048
+L GND #PWR046
 U 1 1 5350563A
 P 1100 2100
-F 0 "#PWR048" H 1100 2100 30  0001 C CNN
+F 0 "#PWR046" H 1100 2100 30  0001 C CNN
 F 1 "GND" H 1100 2030 30  0001 C CNN
 F 2 "" H 1100 2100 60  0000 C CNN
@@
 $EndComp
 $Comp
-L R R16
+L R R15
 U 1 1 53505640
 P 950 1550
-F 0 "R16" V 1030 1550 40  0000 C CNN
+F 0 "R15" V 1030 1550 40  0000 C CNN
 F 1 "10K" V 957 1551 40  0000 C CNN
 F 2 "~" V 880 1550 30  0000 C CNN
@@
 $EndComp
 $Comp
-L GND #PWR049
+L GND #PWR047
 U 1 1 53505646
 P 700 1550
-F 0 "#PWR049" H 700 1550 30  0001 C CNN
+F 0 "#PWR047" H 700 1550 30  0001 C CNN
 F 1 "GND" H 700 1480 30  0001 C CNN
 F 2 "" H 700 1550 60  0000 C CNN
@@
 $EndComp
 $Comp
-L R R17
+L R R16
 U 1 1 537944F7
 P 4000 1100
-F 0 "R17" V 4080 1100 40  0000 C CNN
+F 0 "R16" V 4080 1100 40  0000 C CNN
 F 1 "220R" V 4007 1101 40  0000 C CNN
 F 2 "~" V 3930 1100 30  0000 C CNN
@@
 $EndComp
 $Comp
-L R R18
+L R R17
 U 1 1 53794688
 P 4000 1650
-F 0 "R18" V 4080 1650 40  0000 C CNN
+F 0 "R17" V 4080 1650 40  0000 C CNN
 F 1 "220R" V 4007 1651 40  0000 C CNN
 F 2 "~" V 3930 1650 30  0000 C CNN
@@
 $EndComp
 $Comp
-L R R19
+L R R18
 U 1 1 53794699
 P 4000 2200
-F 0 "R19" V 4080 2200 40  0000 C CNN
+F 0 "R18" V 4080 2200 40  0000 C CNN
 F 1 "220R" V 4007 2201 40  0000 C CNN
 F 2 "~" V 3930 2200 30  0000 C CNN
@@
 $EndComp
 $Comp
-L R R20
+L R R19
 U 1 1 537946AA
 P 4000 2750
-F 0 "R20" V 4080 2750 40  0000 C CNN
+F 0 "R19" V 4080 2750 40  0000 C CNN
 F 1 "220R" V 4007 2751 40  0000 C CNN
 F 2 "~" V 3930 2750 30  0000 C CNN
@@
 $EndComp
 $Comp
-L R R21
+L R R20
 U 1 1 537946BB
 P 4000 3300
-F 0 "R21" V 4080 3300 40  0000 C CNN
+F 0 "R20" V 4080 3300 40  0000 C CNN
 F 1 "220R" V 4007 3301 40  0000 C CNN
 F 2 "~" V 3930 3300 30  0000 C CNN
@@
 $EndComp
 $Comp
-L R R22
+L R R21
 U 1 1 537946CC
 P 4000 3850
-F 0 "R22" V 4080 3850 40  0000 C CNN
+F 0 "R21" V 4080 3850 40  0000 C CNN
 F 1 "220R" V 4007 3851 40  0000 C CNN
 F 2 "~" V 3930 3850 30  0000 C CNN
@@
 $EndComp
 $Comp
-L R R23
+L R R22
 U 1 1 537946FB
 P 4000 4400
-F 0 "R23" V 4080 4400 40  0000 C CNN
+F 0 "R22" V 4080 4400 40  0000 C CNN
 F 1 "220R" V 4007 4401 40  0000 C CNN
 F 2 "~" V 3930 4400 30  0000 C CNN
@@
 $EndComp
 $Comp
-L R R24
+L R R23
 U 1 1 5379470C
 P 4000 4950
-F 0 "R24" V 4080 4950 40  0000 C CNN
+F 0 "R23" V 4080 4950 40  0000 C CNN
 F 1 "220R" V 4007 4951 40  0000 C CNN
 F 2 "~" V 3930 4950 30  0000 C CNN
@@
 	4350 5050 4450 5150
 $Comp
-L GND #PWR050
+L GND #PWR048
 U 1 1 537951D0
 P 5250 5150
-F 0 "#PWR050" H 5250 5150 30  0001 C CNN
+F 0 "#PWR048" H 5250 5150 30  0001 C CNN
 F 1 "GND" H 5250 5080 30  0001 C CNN
 F 2 "" H 5250 5150 60  0000 C CNN

Commit message: MLS800  * Added separated GND : AGND & GND  * Revamped the loops schema  * Put values on all components  * Started to add footprint annotations to some resistors
Parts:
- removed S10, S11, S12, S13, S14, S7, S8, S9: SW_TACT_LED, ~, symbol SW_TACT_LED
- added SW10, SW11, SW12, SW13, SW14, SW15, SW16, SW17: SW_TACT_LED_2, symbol SW_TACT_LED_2
- R15: value 10K -> 1k
Connections:
- net labels added: DGND
- net labels removed: GND
- wire segments 77 -> 61
Other:
- moved on the sheet: R15, R16, R17, R18, R19, R20, R21, R22, R23, U4

Commit message: MLS800  * Started cmp association
Parts:
- renumbered R15 to R17, R16 to R18, R17 to R19, R18 to R20, R19 to R21, R20 to R22, R21 to R23, R22 to R24, R23 to R25, SW16 to SW10, SW17 to SW11, SW10 to SW4, SW11 to SW5, SW12 to SW6, SW13 to SW7, SW14 to SW8, SW15 to SW9
Changed lines of the file:
@@
 Sheet 3 4
 Title ""
-Date "17 aug 2014"
+Date "18 aug 2014"
 Rev ""
 Comp ""
@@
 $EndComp
 $Comp
-L VCC #PWR045
+L VCC #PWR45
 U 1 1 5350562C
 P 2200 1100
-F 0 "#PWR045" H 2200 1200 30  0001 C CNN
+F 0 "#PWR45" H 2200 1200 30  0001 C CNN
 F 1 "VCC" H 2200 1200 30  0000 C CNN
 F 2 "" H 2200 1100 60  0000 C CNN
@@
 $EndComp
 $Comp
-L R R15
+L R R17
 U 1 1 53505640
 P 1000 1550
-F 0 "R15" V 1080 1550 40  0000 C CNN
+F 0 "R17" V 1080 1550 40  0000 C CNN
 F 1 "1k" V 1007 1551 40  0000 C CNN
 F 2 "~" V 930 1550 30  0000 C CNN
@@
 	3250 1850 3350 1950
 $Comp
-L R R16
+L R R18
 U 1 1 537944F7
 P 4050 1100
-F 0 "R16" V 4130 1100 40  0000 C CNN
+F 0 "R18" V 4130 1100 40  0000 C CNN
 F 1 "220R" V 4057 1101 40  0000 C CNN
 F 2 "~" V 3980 1100 30  0000 C CNN
@@
 I2
 $Comp
-L R R17
+L R R19
 U 1 1 53794688
 P 4050 1650
-F 0 "R17" V 4130 1650 40  0000 C CNN
+F 0 "R19" V 4130 1650 40  0000 C CNN
 F 1 "220R" V 4057 1651 40  0000 C CNN
 F 2 "~" V 3980 1650 30  0000 C CNN
@@
 I3
 $Comp
-L R R18
+L R R20
 U 1 1 53794699
 P 4050 2200
-F 0 "R18" V 4130 2200 40  0000 C CNN
+F 0 "R20" V 4130 2200 40  0000 C CNN
 F 1 "220R" V 4057 2201 40  0000 C CNN
 F 2 "~" V 3980 2200 30  0000 C CNN
@@
 I4
 $Comp
-L R R19
+L R R21
 U 1 1 537946AA
 P 4050 2750
-F 0 "R19" V 4130 2750 40  0000 C CNN
+F 0 "R21" V 4130 2750 40  0000 C CNN
 F 1 "220R" V 4057 2751 40  0000 C CNN
 F 2 "~" V 3980 2750 30  0000 C CNN
@@
 I5
 $Comp
-L R R20
+L R R22
 U 1 1 537946BB
 P 4050 3300
-F 0 "R20" V 4130 3300 40  0000 C CNN
+F 0 "R22" V 4130 3300 40  0000 C CNN
 F 1 "220R" V 4057 3301 40  0000 C CNN
 F 2 "~" V 3980 3300 30  0000 C CNN
@@
 I6
 $Comp
-L R R21
+L R R23
 U 1 1 537946CC
 P 4050 3850
-F 0 "R21" V 4130 3850 40  0000 C CNN
+F 0 "R23" V 4130 3850 40  0000 C CNN
 F 1 "220R" V 4057 3851 40  0000 C CNN
 F 2 "~" V 3980 3850 30  0000 C CNN
@@
 I7
 $Comp
-L R R22
+L R R24
 U 1 1 537946FB
 P 4050 4400
-F 0 "R22" V 4130 4400 40  0000 C CNN
+F 0 "R24" V 4130 4400 40  0000 C CNN
 F 1 "220R" V 4057 4401 40  0000 C CNN
 F 2 "~" V 3980 4400 30  0000 C CNN
@@
 I8
 $Comp
-L R R23
+L R R25
 U 1 1 5379470C
 P 4050 4950
-F 0 "R23" V 4130 4950 40  0000 C CNN
+F 0 "R25" V 4130 4950 40  0000 C CNN
 F 1 "220R" V 4057 4951 40  0000 C CNN
 F 2 "~" V 3980 4950 30  0000 C CNN
@@
 	3600 4850 3700 4950
 $Comp
-L SW_TACT_LED_2 SW10
+L SW_TACT_LED_2 SW4
 U 2 1 53B9BB32
 P 4900 1300
-F 0 "SW10" H 4700 1200 60  0000 C CNN
+F 0 "SW4" H 4700 1200 60  0000 C CNN
 F 1 "SW_TACT_LED_2" H 4950 1200 60  0001 C CNN
 F 2 "" H 4900 1300 60  0000 C CNN
@@
 $EndComp
 $Comp
-L SW_TACT_LED_2 SW10
+L SW_TACT_LED_2 SW4
 U 1 1 53B9BB41
 P 4900 1100
-F 0 "SW10" H 4700 1250 60  0000 C CNN
+F 0 "SW4" H 4700 1250 60  0000 C CNN
 F 1 "SW_TACT_LED_2" H 4950 1000 60  0001 C CNN
 F 2 "" H 4900 1100 60  0000 C CNN
@@
 $EndComp
 $Comp
-L SW_TACT_LED_2 SW11
+L SW_TACT_LED_2 SW5
 U 2 1 53B9BB96
 P 4900 1850
-F 0 "SW11" H 4700 1750 60  0000 C CNN
+F 0 "SW5" H 4700 1750 60  0000 C CNN
 F 1 "SW_TACT_LED_2" H 4950 1750 60  0001 C CNN
 F 2 "" H 4900 1850 60  0000 C CNN
@@
 $EndComp
 $Comp
-L SW_TACT_LED_2 SW11
+L SW_TACT_LED_2 SW5
 U 1 1 53B9BB9C
 P 4900 1650
-F 0 "SW11" H 4700 1800 60  0000 C CNN
+F 0 "SW5" H 4700 1800 60  0000 C CNN
 F 1 "SW_TACT_LED_2" H 4950 1550 60  0001 C CNN
 F 2 "" H 4900 1650 60  0000 C CNN
@@
 $EndComp
 $Comp
-L SW_TACT_LED_2 SW12
+L SW_TACT_LED_2 SW6
 U 2 1 53B9BBAC
 P 4900 2400
-F 0 "SW12" H 4700 2300 60  0000 C CNN
+F 0 "SW6" H 4700 2300 60  0000 C CNN
 F 1 "SW_TACT_LED_2" H 4950 2300 60  0001 C CNN
 F 2 "" H 4900 2400 60  0000 C CNN
@@
 $EndComp
 $Comp
-L SW_TACT_LED_2 SW12
+L SW_TACT_LED_2 SW6
 U 1 1 53B9BBB2
 P 4900 2200
-F 0 "SW12" H 4700 2350 60  0000 C CNN
+F 0 "SW6" H 4700 2350 60  0000 C CNN
 F 1 "SW_TACT_LED_2" H 4950 2100 60  0001 C CNN
 F 2 "" H 4900 2200 60  0000 C CNN
@@
 $EndComp
 $Comp
-L SW_TACT_LED_2 SW13
+L SW_TACT_LED_2 SW7
 U 2 1 53B9BBB8
 P 4900 2950
-F 0 "SW13" H 4700 2850 60  0000 C CNN
+F 0 "SW7" H 4700 2850 60  0000 C CNN
 F 1 "SW_TACT_LED_2" H 4950 2850 60  0001 C CNN
 F 2 "" H 4900 2950 60  0000 C CNN
@@
 $EndComp
 $Comp
-L SW_TACT_LED_2 SW13
+L SW_TACT_LED_2 SW7
 U 1 1 53B9BBBE
 P 4900 2750
-F 0 "SW13" H 4700 2900 60  0000 C CNN
+F 0 "SW7" H 4700 2900 60  0000 C CNN
 F 1 "SW_TACT_LED_2" H 4950 2650 60  0001 C CNN
 F 2 "" H 4900 2750 60  0000 C CNN
@@
 $EndComp
 $Comp
-L SW_TACT_LED_2 SW14
+L SW_TACT_LED_2 SW8
 U 2 1 53B9BBC4
 P 4900 3500
-F 0 "SW14" H 4700 3400 60  0000 C CNN
+F 0 "SW8" H 4700 3400 60  0000 C CNN
 F 1 "SW_TACT_LED_2" H 4950 3400 60  0001 C CNN
 F 2 "" H 4900 3500 60  0000 C CNN
@@
 $EndComp
 $Comp
-L SW_TACT_LED_2 SW14
+L SW_TACT_LED_2 SW8
 U 1 1 53B9BBCA
 P 4900 3300
-F 0 "SW14" H 4700 3450 60  0000 C CNN
+F 0 "SW8" H 4700 3450 60  0000 C CNN
 F 1 "SW_TACT_LED_2" H 4950 3200 60  0001 C CNN
 F 2 "" H 4900 3300 60  0000 C CNN
@@
 $EndComp
 $Comp
-L SW_TACT_LED_2 SW15
+L SW_TACT_LED_2 SW9
 U 2 1 53B9BBD0
 P 4900 4050
-F 0 "SW15" H 4700 3950 60  0000 C CNN
+F 0 "SW9" H 4700 3950 60  0000 C CNN
 F 1 "SW_TACT_LED_2" H 4950 3950 60  0001 C CNN
 F 2 "" H 4900 4050 60  0000 C CNN
@@
 $EndComp
 $Comp
-L SW_TACT_LED_2 SW15
+L SW_TACT_LED_2 SW9
 U 1 1 53B9BBD6
 P 4900 3850
-F 0 "SW15" H 4700 4000 60  0000 C CNN
+F 0 "SW9" H 4700 4000 60  0000 C CNN
 F 1 "SW_TACT_LED_2" H 4950 3750 60  0001 C CNN
 F 2 "" H 4900 3850 60  0000 C CNN
@@
 $EndComp
 $Comp
-L SW_TACT_LED_2 SW16
+L SW_TACT_LED_2 SW10
 U 2 1 53B9BBDC
 P 4900 4600
-F 0 "SW16" H 4700 4500 60  0000 C CNN
+F 0 "SW10" H 4700 4500 60  0000 C CNN
 F 1 "SW_TACT_LED_2" H 4950 4500 60  0001 C CNN
 F 2 "" H 4900 4600 60  0000 C CNN
@@
 $EndComp
 $Comp
-L SW_TACT_LED_2 SW16
+L SW_TACT_LED_2 SW10
 U 1 1 53B9BBE2
 P 4900 4400
-F 0 "SW16" H 4700 4550 60  0000 C CNN
+F 0 "SW10" H 4700 4550 60  0000 C CNN
 F 1 "SW_TACT_LED_2" H 4950 4300 60  0001 C CNN
 F 2 "" H 4900 4400 60  0000 C CNN
@@
 $EndComp
 $Comp
-L SW_TACT_LED_2 SW17
+L SW_TACT_LED_2 SW11
 U 2 1 53B9BBE8
 P 4900 5150
-F 0 "SW17" H 4700 5050 60  0000 C CNN
+F 0 "SW11" H 4700 5050 60  0000 C CNN
 F 1 "SW_TACT_LED_2" H 4950 5050 60  0001 C CNN
 F 2 "" H 4900 5150 60  0000 C CNN
@@
 $EndComp
 $Comp
-L SW_TACT_LED_2 SW17
+L SW_TACT_LED_2 SW11
 U 1 1 53B9BBEE
 P 4900 4950
-F 0 "SW17" H 4700 5100 60  0000 C CNN
+F 0 "SW11" H 4700 5100 60  0000 C CNN
 F 1 "SW_TACT_LED_2" H 4950 4850 60  0001 C CNN
 F 2 "" H 4900 4950 60  0000 C CNN
@@
 Connection ~ 5250 1300
 $Comp
-L DGND #PWR046
+L DGND #PWR47
 U 1 1 53F19F43
 P 5250 5350
-F 0 "#PWR046" H 5250 5350 40  0001 C CNN
+F 0 "#PWR47" H 5250 5350 40  0001 C CNN
 F 1 "DGND" H 5250 5280 40  0000 C CNN
 F 2 "" H 5250 5350 60  0000 C CNN
@@
 $EndComp
 $Comp
-L DGND #PWR047
+L DGND #PWR46
 U 1 1 53F19F5C
 P 2200 3800
-F 0 "#PWR047" H 2200 3800 40  0001 C CNN
+F 0 "#PWR46" H 2200 3800 40  0001 C CNN
 F 1 "DGND" H 2200 3730 40  0000 C CNN
 F 2 "" H 2200 3800 60  0000 C CNN
@@
 $EndComp
 $Comp
-L DGND #PWR048
+L DGND #PWR44
 U 1 1 53F19F6B
 P 1100 2100
-F 0 "#PWR048" H 1100 2100 40  0001 C CNN
+F 0 "#PWR44" H 1100 2100 40  0001 C CNN
 F 1 "DGND" H 1100 2030 40  0000 C CNN
 F 2 "" H 1100 2100 60  0000 C CNN
@@
 $EndComp
 $Comp
-L DGND #PWR049
+L DGND #PWR43
 U 1 1 53F19F7A
 P 750 1550
-F 0 "#PWR049" H 750 1550 40  0001 C CNN
+F 0 "#PWR43" H 750 1550 40  0001 C CNN
 F 1 "DGND" H 750 1480 40  0000 C CNN
 F 2 "" H 750 1550 60  0000 C CNN

Commit message: MLS800 :  - assigning footprints
Parts:
- R17, R18, R19, R20, R21, R22, R23, R24, R25: footprint ~ -> Resistors_SMD:R_0805_HandSoldering
- U4: footprint MODULE -> Housings_SSOP:SSOP-28
Changed lines of the file:
@@
 F 0 "U4" H 1650 3550 50  0000 C CNN
 F 1 "MCP23017" H 2650 1350 50  0000 C CNN
-F 2 "MODULE" H 1700 1350 50  0001 C CNN
+F 2 "Housings_SSOP:SSOP-28" H 1700 1350 50  0001 C CNN
 F 3 "DOCUMENTATION" H 2200 2400 50  0001 C CNN
 	1    2200 2450
@@
 F 0 "R17" V 1080 1550 40  0000 C CNN
 F 1 "1k" V 1007 1551 40  0000 C CNN
-F 2 "~" V 930 1550 30  0000 C CNN
+F 2 "Resistors_SMD:R_0805_HandSoldering" V 930 1550 30  0001 C CNN
 F 3 "~" H 1000 1550 30  0000 C CNN
 	1    1000 1550
@@
 F 0 "R18" V 4130 1100 40  0000 C CNN
 F 1 "220R" V 4057 1101 40  0000 C CNN
-F 2 "~" V 3980 1100 30  0000 C CNN
+F 2 "Resistors_SMD:R_0805_HandSoldering" V 3980 1100 30  0001 C CNN
 F 3 "~" H 4050 1100 30  0000 C CNN
 	1    4050 1100
@@
 F 0 "R19" V 4130 1650 40  0000 C CNN
 F 1 "220R" V 4057 1651 40  0000 C CNN
-F 2 "~" V 3980 1650 30  0000 C CNN
+F 2 "Resistors_SMD:R_0805_HandSoldering" V 3980 1650 30  0001 C CNN
 F 3 "~" H 4050 1650 30  0000 C CNN
 	1    4050 1650
@@
 F 0 "R20" V 4130 2200 40  0000 C CNN
 F 1 "220R" V 4057 2201 40  0000 C CNN
-F 2 "~" V 3980 2200 30  0000 C CNN
+F 2 "Resistors_SMD:R_0805_HandSoldering" V 3980 2200 30  0001 C CNN
 F 3 "~" H 4050 2200 30  0000 C CNN
 	1    4050 2200
@@
 F 0 "R21" V 4130 2750 40  0000 C CNN
 F 1 "220R" V 4057 2751 40  0000 C CNN
-F 2 "~" V 3980 2750 30  0000 C CNN
+F 2 "Resistors_SMD:R_0805_HandSoldering" V 3980 2750 30  0001 C CNN
 F 3 "~" H 4050 2750 30  0000 C CNN
 	1    4050 2750
@@
 F 0 "R22" V 4130 3300 40  0000 C CNN
 F 1 "220R" V 4057 3301 40  0000 C CNN
-F 2 "~" V 3980 3300 30  0000 C CNN
+F 2 "Resistors_SMD:R_0805_HandSoldering" V 3980 3300 30  0001 C CNN
 F 3 "~" H 4050 3300 30  0000 C CNN
 	1    4050 3300
@@
 F 0 "R23" V 4130 3850 40  0000 C CNN
 F 1 "220R" V 4057 3851 40  0000 C CNN
-F 2 "~" V 3980 3850 30  0000 C CNN
+F 2 "Resistors_SMD:R_0805_HandSoldering" V 3980 3850 30  0001 C CNN
 F 3 "~" H 4050 3850 30  0000 C CNN
 	1    4050 3850
@@
 F 0 "R24" V 4130 4400 40  0000 C CNN
 F 1 "220R" V 4057 4401 40  0000 C CNN
-F 2 "~" V 3980 4400 30  0000 C CNN
+F 2 "Resistors_SMD:R_0805_HandSoldering" V 3980 4400 30  0001 C CNN
 F 3 "~" H 4050 4400 30  0000 C CNN
 	1    4050 4400
@@
 F 0 "R25" V 4130 4950 40  0000 C CNN
 F 1 "220R" V 4057 4951 40  0000 C CNN
-F 2 "~" V 3980 4950 30  0000 C CNN
+F 2 "Resistors_SMD:R_0805_HandSoldering" V 3980 4950 30  0001 C CNN
 F 3 "~" H 4050 4950 30  0000 C CNN
 	1    4050 4950
