File: mls800_front_panel.sch (KiCad schematic (older format))
At the start: 0 parts

Commit message: MLS800 : added LTC-5723HR  to custom-display library
MLS800 : fixed AS1115 pin placement to match main grid
Parts:
- added AFF?: LTC-5723HR, symbol LTC-5723HR
- added R?: R, symbol R
- added U?: AS1115, MODULE, symbol AS1115
Connections:
- new net: R?.1, U?.13 (ISET)
- new net DGND: U?.6 (GND)
- new net DIG1: AFF?.12 (D1), U?.2 (DIG0)
- new net DIG2: AFF?.9 (D2), U?.3 (DIG1)
- new net DIG3: AFF?.8 (D3), U?.4 (DIG2)
- new net DIG4: AFF?.6 (D4), U?.5 (DIG3)
- new net IRQ: U?.24 (IRQ)
- new net SCL: U?.14 (SCL)
- new net SDA: U?.1 (SDA)
- new net SEGA: AFF?.11 (a), U?.15 (SEGA)
- new net SEGB: AFF?.7 (b), U?.17 (SEGB)
- new net SEGC: AFF?.4 (c), U?.20 (SEGC)
- new net SEGD: AFF?.2 (d), U?.23 (SEGD)
- new net SEGDP: AFF?.3 (dp), U?.22 (SEGDP)
- new net SEGE: AFF?.1 (e), U?.21 (SEGE)
- new net SEGF: AFF?.10 (f), U?.16 (SEGF)
- new net SEGG: AFF?.5 (g), U?.18 (SEGG)
- new net VCC: R?.2, U?.19 (VDD)
Changed lines of the file:
@@
 LIBS:custom-conn
 LIBS:custom-device
+LIBS:custom-display
 LIBS:mls800-cache
 EELAYER 24 0
@@
 Comment4 ""
 $EndDescr
+$Comp
+L LTC-5723HR AFF?
+U 1 1 543EEF72
+P 6050 2250
+F 0 "AFF?" H 5450 2700 60  0000 C CNN
+F 1 "LTC-5723HR" H 5550 1800 60  0000 C CNN
+F 2 "" H 5550 2250 60  0000 C CNN
+F 3 "" H 5550 2250 60  0000 C CNN
+	1    6050 2250
+	1    0    0    -1
+$EndComp
+$Comp
+L AS1115 U?
+U 1 1 543EEFD5
+P 2500 1900
+F 0 "U?" H 1950 3000 50  0000 C CNN
+F 1 "AS1115" H 2950 800 50  0000 C CNN
+F 2 "MODULE" H 2000 800 50  0001 C CNN
+F 3 "DOCUMENTATION" H 2500 1850 50  0001 C CNN
+	1    2500 1900
+	1    0    0    -1
+$EndComp
+Entry Wire Line
+	3650 1000 3750 1100
+Entry Wire Line
+	3650 1100 3750 1200
+Entry Wire Line
+	3650 1200 3750 1300
+Entry Wire Line
+	3650 1300 3750 1400
+Text Label 3450 1000 0    60   ~ 0
+DIG1
+Text Label 3450 1100 0    60   ~ 0
+DIG2
+Text Label 3450 1200 0    60   ~ 0
+DIG3
+Text Label 3450 1300 0    60   ~ 0
+DIG4
+Text Label 7450 2100 0    60   ~ 0
+DIG1
+Text Label 7450 2200 0    60   ~ 0
+DIG2
+Entry Wire Line
+	7650 2100 7750 2200
+Entry Wire Line
+	7650 2200 7750 2300
+Entry Wire Line
+	7650 2300 7750 2400
+Entry Wire Line
+	7650 2400 7750 2500
+Text Label 7450 2300 0    60   ~ 0
+DIG3
+Text Label 7450 2400 0    60   ~ 0
+DIG4
+Entry Wire Line
+	3750 1850 3850 1950
+Entry Wire Line
+	3750 1950 3850 2050
+Entry Wire Line
+	3750 2050 3850 2150
+Entry Wire Line
+	3750 2150 3850 2250
+Entry Wire Line
+	3750 2250 3850 2350
+Entry Wire Line
+	3750 2350 3850 2450
+Entry Wire Line
+	3750 2450 3850 2550
+Entry Wire Line
+	3750 2550 3850 2650
+Text Label 3450 1850 0    60   ~ 0
+SEGA
+Text Label 3450 1950 0    60   ~ 0
+SEGB
+Text Label 3450 2050 0    60   ~ 0
+SEGC
+Text Label 3450 2150 0    60   ~ 0
+SEGD
+Text Label 3450 2250 0    60   ~ 0
+SEGE
+Text Label 3450 2350 0    60   ~ 0
+SEGF
+Text Label 3450 2450 0    60   ~ 0
+SEGG
+Text Label 3450 2550 0    60   ~ 0
+SEGDP
+Text Label 4600 1900 2    60   ~ 0
+SEGA
+Text Label 4600 2000 2    60   ~ 0
+SEGB
+Text Label 4600 2100 2    60   ~ 0
+SEGC
+Text Label 4600 2200 2    60   ~ 0
+SEGD
+Text Label 4600 2300 2    60   ~ 0
+SEGE
+Text Label 4600 2400 2    60   ~ 0
+SEGF
+Text Label 4600 2500 2    60   ~ 0
+SEGG
+Text Label 4600 2600 2    60   ~ 0
+SEGDP
+Entry Wire Line
+	4200 1800 4300 1900
+Entry Wire Line
+	4200 1900 4300 2000
+Entry Wire Line
+	4200 2000 4300 2100
+Entry Wire Line
+	4200 2100 4300 2200
+Entry Wire Line
+	4200 2200 4300 2300
+Entry Wire Line
+	4200 2300 4300 2400
+Entry Wire Line
+	4200 2400 4300 2500
+Entry Wire Line
+	4200 2500 4300 2600
+Wire Wire Line
+	3650 1000 3450 1000
+Wire Wire Line
+	3450 1100 3650 1100
+Wire Wire Line
+	3650 1200 3450 1200
+Wire Wire Line
+	3450 1300 3650 1300
+Wire Wire Line
+	7650 2400 7450 2400
+Wire Wire Line
+	7650 2300 7450 2300
+Wire Wire Line
+	7650 2200 7450 2200
+Wire Wire Line
+	7650 2100 7450 2100
+Wire Wire Line
+	3750 2550 3450 2550
+Wire Wire Line
+	3450 2450 3750 2450
+Wire Wire Line
+	3750 2350 3450 2350
+Wire Wire Line
+	3450 2250 3750 2250
+Wire Wire Line
+	3750 2150 3450 2150
+Wire Wire Line
+	3750 2050 3450 2050
+Wire Wire Line
+	3450 1950 3750 1950
+Wire Wire Line
+	3750 1850 3450 1850
+Wire Wire Line
+	4600 2600 4300 2600
+Wire Wire Line
+	4300 2500 4600 2500
+Wire Wire Line
+	4600 2400 4300 2400
+Wire Wire Line
+	4300 2300 4600 2300
+Wire Wire Line
+	4600 2200 4300 2200
+Wire Wire Line
+	4600 2100 4300 2100
+Wire Wire Line
+	4300 2000 4600 2000
+Wire Wire Line
+	4600 1900 4300 1900
+Wire Bus Line
+	3850 1950 3850 2650
+Wire Bus Line
+	3850 2650 4200 2650
+Wire Bus Line
+	4200 2650 4200 1800
+Wire Bus Line
+	3750 1100 3750 1700
+Wire Bus Line
+	3750 1700 7750 1700
+Wire Bus Line
+	7750 1700 7750 2500
+$Comp
+L VCC #PWR?
+U 1 1 543F0201
+P 1050 950
+F 0 "#PWR?" H 1050 1050 30  0001 C CNN
+F 1 "VCC" H 1050 1050 30  0000 C CNN
+F 2 "" H 1050 950 60  0000 C CNN
+F 3 "" H 1050 950 60  0000 C CNN
+	1    1050 950
+	0    -1   -1   0
+$EndComp
+$Comp
+L DGND #PWR?
+U 1 1 543F021F
+P 2500 3250
+F 0 "#PWR?" H 2500 3250 40  0001 C CNN
+F 1 "DGND" H 2500 3180 40  0000 C CNN
+F 2 "" H 2500 3250 60  0000 C CNN
+F 3 "" H 2500 3250 60  0000 C CNN
+	1    2500 3250
+	1    0    0    -1
+$EndComp
+Text HLabel 1550 2400 0    60   Input ~ 0
+SDA
+Text HLabel 1550 2500 0    60   Input ~ 0
+SCL
+Text HLabel 1550 2600 0    60   Input ~ 0
+IRQ
+$Comp
+L R R?
+U 1 1 543F1E5E
+P 1300 1050
+F 0 "R?" V 1380 1050 40  0000 C CNN
+F 1 "R" V 1307 1051 40  0000 C CNN
+F 2 "" V 1230 1050 30  0000 C CNN
+F 3 "" H 1300 1050 30  0000 C CNN
+	1    1300 1050
+	0    1    1    0
+$EndComp
+Wire Wire Line
+	1050 1050 1050 950
+Wire Wire Line
+	1050 950  1550 950
 $EndSCHEMATC

Commit message: MLS800 : fixed broken layout
MLS800 : added some comments on schematics rather than using a notepad :)
Parts:
- added R?: 1K, symbol R
- added SW? (x3): SW_TACT_LED, symbol SW_TACT_LED
- added U?: MCP23017, MODULE, symbol MCP23017
Connections:
- net DGND: now also U?.10 (VSS)
- net VCC: now also R?.2, U?.9 (VDD)
- new net: R?.1, U?.18 (~RESET)
- new net led1_a: U?.21 (GPA0)
Other:
- note added: "Bi color leds : which button cap to get ?\n - Can't take the transparent red one or green led could be "ugly"\n - Transparent white could be ugly on its own..."
- note added: "Rset : \n - 20 mA : 22.6k\n - 30 mA : 14.7k\n - 40 mA : 10.84k"
- note added: "With single color leds, AS1115 can drive the loops state leds. This eliminate the needs of an additionnal MCP23017.\nThe button led resistances needs to be adjusted though (an additionnal resistance for each led ?)"
Changed lines of the file:
@@
 Wire Wire Line
 	1050 950  1550 950
+$Comp
+L SW_TACT_LED SW?
+U 1 1 543F13D1
+P 4700 4350
+F 0 "SW?" H 4500 4500 60  0000 C CNN
+F 1 "SW_TACT_LED" H 4670 4250 60  0001 C CNN
+F 2 "" H 4700 4350 60  0000 C CNN
+F 3 "" H 4700 4350 60  0000 C CNN
+	1    4700 4350
+	1    0    0    -1
+$EndComp
+$Comp
+L SW_TACT_LED SW?
+U 2 1 543F13EA
+P 4700 4600
+F 0 "SW?" H 4500 4750 60  0000 C CNN
+F 1 "SW_TACT_LED" H 4670 4500 60  0001 C CNN
+F 2 "" H 4700 4600 60  0000 C CNN
+F 3 "" H 4700 4600 60  0000 C CNN
+	2    4700 4600
+	1    0    0    -1
+$EndComp
+$Comp
+L SW_TACT_LED SW?
+U 3 1 543F145D
+P 4700 4900
+F 0 "SW?" H 4500 5050 60  0000 C CNN
+F 1 "SW_TACT_LED" H 4670 4800 60  0001 C CNN
+F 2 "" H 4700 4900 60  0000 C CNN
+F 3 "" H 4700 4900 60  0000 C CNN
+	3    4700 4900
+	1    0    0    -1
+$EndComp
+$Comp
+L MCP23017 U?
+U 1 1 543F149E
+P 2500 5250
+F 0 "U?" H 1950 6350 50  0000 C CNN
+F 1 "MCP23017" H 2950 4150 50  0000 C CNN
+F 2 "MODULE" H 2000 4150 50  0001 C CNN
+F 3 "DOCUMENTATION" H 2500 5200 50  0001 C CNN
+	1    2500 5250
+	1    0    0    -1
+$EndComp
+$Comp
+L DGND #PWR?
+U 1 1 543F1572
+P 2500 6600
+F 0 "#PWR?" H 2500 6600 40  0001 C CNN
+F 1 "DGND" H 2500 6530 40  0000 C CNN
+F 2 "" H 2500 6600 60  0000 C CNN
+F 3 "" H 2500 6600 60  0000 C CNN
+	1    2500 6600
+	1    0    0    -1
+$EndComp
+$Comp
+L R R?
+U 1 1 543F18A9
+P 1300 4400
+F 0 "R?" V 1380 4400 40  0000 C CNN
+F 1 "1K" V 1307 4401 40  0000 C CNN
+F 2 "" V 1230 4400 30  0000 C CNN
+F 3 "" H 1300 4400 30  0000 C CNN
+	1    1300 4400
+	0    1    1    0
+$EndComp
+$Comp
+L VCC #PWR?
+U 1 1 543F1932
+P 1050 4300
+F 0 "#PWR?" H 1050 4400 30  0001 C CNN
+F 1 "VCC" H 1050 4400 30  0000 C CNN
+F 2 "" H 1050 4300 60  0000 C CNN
+F 3 "" H 1050 4300 60  0000 C CNN
+	1    1050 4300
+	0    -1   -1   0
+$EndComp
+Wire Wire Line
+	1050 4300 1550 4300
+Wire Wire Line
+	1050 4400 1050 4300
+Text Notes 850  1550 0    60   ~ 0
+Rset : \n - 20 mA : 22.6k\n - 30 mA : 14.7k\n - 40 mA : 10.84k
+Text Notes 2150 3950 0    60   ~ 0
+Bi color leds : which button cap to get ?\n - Can't take the transparent red one or green led could be "ugly"\n - Transparent white could be ugly on its own...
+Text Label 3450 4350 0    60   ~ 0
+led1_a
+Text Notes 5850 3900 0    60   ~ 0
+With single color leds, AS1115 can drive the loops state leds. This eliminate the needs of an additionnal MCP23017.\nThe button led resistances needs to be adjusted though (an additionnal resistance for each led ?)
 $EndSCHEMATC

Commit message: MLS800 : disabled switch tact led "interchangeable" units => fixed annotations
MLS800 : front panel schematic seems to be completed
Parts:
- removed R?: 1K, symbol R
- removed SW? (x3): SW_TACT_LED, symbol SW_TACT_LED
- removed U?: MCP23017, MODULE, symbol MCP23017
- added R28, R29, R30, R31, R32, R33, R34, R35: 110R, symbol R
- added SW10, SW11, SW12, SW13, SW14, SW15, SW16, SW17, SW9: SW_TACT_LED, symbol SW_TACT_LED
- gave numbers to parts that had none: 3
Connections:
- net SEGA: now also R28.2, SW9.4
- net SEGB: now also R29.2, SW10.4
- net SEGC: now also R30.2, SW11.4
- net SEGD: now also R31.2, SW12.4
- net SEGDP: now also R35.2, SW16.4
- net SEGE: now also R32.2, SW13.4
- net SEGF: now also R33.2, SW14.4
- net SEGG: now also R34.2, SW15.4
- net LEDS: now reaches U6.7 (DIG4)
- net LEDS: now also SW10.2, SW11.2, SW12.2, SW13.2, SW14.2, SW15.2, SW16.2, SW17.2
- new net: SW10.1, SW11.1, SW12.1, SW13.1, SW14.1, SW15.1, SW16.1, SW9.1, U6.20 (SEGC)
- new net: R28.1, SW10.3
- new net: R29.1, SW11.3
- new net: R30.1, SW12.3
- new net: R31.1, SW13.3
- new net: R32.1, SW14.3
- new net: R33.1, SW15.3
- new net: R34.1, SW16.3
- new net: R35.1, SW17.3
- no-connect marks 0 -> 3
Other:
- note added: "Si 5GH, pour 5V : \n - Green : Foward Voltage = 2.2V => 2.8V => R = 112R\n - Red : Foward Voltage = 2V => 3V => R = 110R\n\nAu choix Rled = 100R ou 110R suivant le résultat des tests"

Commit message: MLS800 : disabled switch tact led "interchangeable" units => fixed annotations
MLS800 : fixed some erc errors in old "misc" sheet
Parts:
- renumbered SW9 to SW12, SW10 to SW12, SW10 to SW13, SW11 to SW13, SW11 to SW14, SW12 to SW14, SW12 to SW15, SW13 to SW15, SW13 to SW16, SW14 to SW16, SW14 to SW17, SW15 to SW17, SW15 to SW18, SW16 to SW18, SW16 to SW19, SW17 to SW19
Changed lines of the file:
@@
 	3750 1700 7750 1700
 $Comp
-L VCC #PWR101
+L VCC #PWR0103
 U 1 1 543F0201
 P 1050 950
-F 0 "#PWR101" H 1050 1050 30  0001 C CNN
+F 0 "#PWR0103" H 1050 1050 30  0001 C CNN
 F 1 "VCC" H 1050 1050 30  0000 C CNN
 F 2 "" H 1050 950 60  0000 C CNN
@@
 $EndComp
 $Comp
-L DGND #PWR102
+L DGND #PWR0104
 U 1 1 543F021F
 P 2500 3250
-F 0 "#PWR102" H 2500 3250 40  0001 C CNN
+F 0 "#PWR0104" H 2500 3250 40  0001 C CNN
 F 1 "DGND" H 2500 3180 40  0000 C CNN
 F 2 "" H 2500 3250 60  0000 C CNN
@@
 With single color leds, AS1115 can drive the loops state leds. This eliminate the needs of an additionnal MCP23017.\nThe button led resistances needs to be adjusted though (an additionnal resistance for each led ?)
 $Comp
-L SW_TACT_LED SW9
+L SW_TACT_LED SW12
 U 1 1 54402E3F
 P 4750 3550
-F 0 "SW9" H 4550 3700 60  0000 C CNN
+F 0 "SW12" H 4550 3700 60  0000 C CNN
 F 1 "SW_TACT_LED" H 4720 3450 60  0001 C CNN
 F 2 "" H 4750 3550 60  0000 C CNN
@@
 $EndComp
 $Comp
-L SW_TACT_LED SW10
+L SW_TACT_LED SW13
 U 1 1 54402F2D
 P 4750 3800
-F 0 "SW10" H 4550 3950 60  0000 C CNN
+F 0 "SW13" H 4550 3950 60  0000 C CNN
 F 1 "SW_TACT_LED" H 4720 3700 60  0001 C CNN
 F 2 "" H 4750 3800 60  0000 C CNN
@@
 $EndComp
 $Comp
-L SW_TACT_LED SW11
+L SW_TACT_LED SW14
 U 1 1 54402F4E
 P 4750 4050
-F 0 "SW11" H 4550 4200 60  0000 C CNN
+F 0 "SW14" H 4550 4200 60  0000 C CNN
 F 1 "SW_TACT_LED" H 4720 3950 60  0001 C CNN
 F 2 "" H 4750 4050 60  0000 C CNN
@@
 $EndComp
 $Comp
-L SW_TACT_LED SW12
+L SW_TACT_LED SW15
 U 1 1 54402F70
 P 4750 4300
-F 0 "SW12" H 4550 4450 60  0000 C CNN
+F 0 "SW15" H 4550 4450 60  0000 C CNN
 F 1 "SW_TACT_LED" H 4720 4200 60  0001 C CNN
 F 2 "" H 4750 4300 60  0000 C CNN
@@
 $EndComp
 $Comp
-L SW_TACT_LED SW13
+L SW_TACT_LED SW16
 U 1 1 54402F97
 P 4750 4550
-F 0 "SW13" H 4550 4700 60  0000 C CNN
+F 0 "SW16" H 4550 4700 60  0000 C CNN
 F 1 "SW_TACT_LED" H 4720 4450 60  0001 C CNN
 F 2 "" H 4750 4550 60  0000 C CNN
@@
 $EndComp
 $Comp
-L SW_TACT_LED SW14
+L SW_TACT_LED SW17
 U 1 1 54403051
 P 4750 4800
-F 0 "SW14" H 4550 4950 60  0000 C CNN
+F 0 "SW17" H 4550 4950 60  0000 C CNN
 F 1 "SW_TACT_LED" H 4720 4700 60  0001 C CNN
 F 2 "" H 4750 4800 60  0000 C CNN
@@
 $EndComp
 $Comp
-L SW_TACT_LED SW15
+L SW_TACT_LED SW18
 U 1 1 54403086
 P 4750 5050
-F 0 "SW15" H 4550 5200 60  0000 C CNN
+F 0 "SW18" H 4550 5200 60  0000 C CNN
 F 1 "SW_TACT_LED" H 4720 4950 60  0001 C CNN
 F 2 "" H 4750 5050 60  0000 C CNN
@@
 $EndComp
 $Comp
-L SW_TACT_LED SW16
+L SW_TACT_LED SW19
 U 1 1 544030B0
 P 4750 5300
-F 0 "SW16" H 4550 5450 60  0000 C CNN
+F 0 "SW19" H 4550 5450 60  0000 C CNN
 F 1 "SW_TACT_LED" H 4720 5200 60  0001 C CNN
 F 2 "" H 4750 5300 60  0000 C CNN
@@
 	5050 3550 5050 5500
 Wire Wire Line
-	3750 5500 5050 5500
-Wire Wire Line
-	3750 2700 3750 5500
+	5050 5500 3750 5500
+Wire Wire Line
+	3750 5500 3750 2700
 Wire Wire Line
 	3750 2700 3450 2700
@@
 	4050 2750 4050 5200
 $Comp
-L SW_TACT_LED SW10
+L SW_TACT_LED SW12
 U 2 1 54405D5F
 P 6850 3550
-F 0 "SW10" H 6650 3700 60  0000 C CNN
+F 0 "SW12" H 6650 3700 60  0000 C CNN
 F 1 "SW_TACT_LED" H 6820 3450 60  0001 C CNN
 F 2 "" H 6850 3550 60  0000 C CNN
@@
 $EndComp
 $Comp
-L SW_TACT_LED SW11
+L SW_TACT_LED SW13
 U 2 1 54405E2B
 P 6850 3800
-F 0 "SW11" H 6650 3950 60  0000 C CNN
+F 0 "SW13" H 6650 3950 60  0000 C CNN
 F 1 "SW_TACT_LED" H 6820 3700 60  0001 C CNN
 F 2 "" H 6850 3800 60  0000 C CNN
@@
 $EndComp
 $Comp
-L SW_TACT_LED SW12
+L SW_TACT_LED SW14
 U 2 1 54405E54
 P 6850 4050
-F 0 "SW12" H 6650 4200 60  0000 C CNN
+F 0 "SW14" H 6650 4200 60  0000 C CNN
 F 1 "SW_TACT_LED" H 6820 3950 60  0001 C CNN
 F 2 "" H 6850 4050 60  0000 C CNN
@@
 $EndComp
 $Comp
-L SW_TACT_LED SW13
+L SW_TACT_LED SW15
 U 2 1 54405E7E
 P 6850 4300
-F 0 "SW13" H 6650 4450 60  0000 C CNN
+F 0 "SW15" H 6650 4450 60  0000 C CNN
 F 1 "SW_TACT_LED" H 6820 4200 60  0001 C CNN
 F 2 "" H 6850 4300 60  0000 C CNN
@@
 $EndComp
 $Comp
-L SW_TACT_LED SW14
+L SW_TACT_LED SW16
 U 2 1 54405EA9
 P 6850 4550
-F 0 "SW14" H 6650 4700 60  0000 C CNN
+F 0 "SW16" H 6650 4700 60  0000 C CNN
 F 1 "SW_TACT_LED" H 6820 4450 60  0001 C CNN
 F 2 "" H 6850 4550 60  0000 C CNN
@@
 $EndComp
 $Comp
-L SW_TACT_LED SW15
+L SW_TACT_LED SW17
 U 2 1 54405ED5
 P 6850 4800
-F 0 "SW15" H 6650 4950 60  0000 C CNN
+F 0 "SW17" H 6650 4950 60  0000 C CNN
 F 1 "SW_TACT_LED" H 6820 4700 60  0001 C CNN
 F 2 "" H 6850 4800 60  0000 C CNN
@@
 $EndComp
 $Comp
-L SW_TACT_LED SW16
+L SW_TACT_LED SW18
 U 2 1 54405F27
 P 6850 5050
-F 0 "SW16" H 6650 5200 60  0000 C CNN
+F 0 "SW18" H 6650 5200 60  0000 C CNN
 F 1 "SW_TACT_LED" H 6820 4950 60  0001 C CNN
 F 2 "" H 6850 5050 60  0000 C CNN
@@
 $EndComp
 $Comp
-L SW_TACT_LED SW17
+L SW_TACT_LED SW19
 U 2 1 54405F59
 P 6850 5300
-F 0 "SW17" H 6650 5450 60  0000 C CNN
+F 0 "SW19" H 6650 5450 60  0000 C CNN
 F 1 "SW_TACT_LED" H 6820 5200 60  0001 C CNN
 F 2 "" H 6850 5300 60  0000 C CNN

Commit message: MLS800
* updated layout to match AS1115 diagrams
* added pull-up resistors
* removed useless sheets
Parts:
- added SW20, SW21: SW_TACT_LED, symbol SW_TACT_LED
Connections:
- net SEGE: now also SW20.4
- net SEGF: now also SW21.4
- net at SW12.1, SW13.1, SW14.1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: now also U6.19 (VDD); no longer U6.20 (SEGC)
- new net: SW20.1, SW21.1, U6.20 (SEGC)
Changed lines of the file:
@@
 $Descr A4 11693 8268
 encoding utf-8
-Sheet 5 5
+Sheet 4 3
 Title ""
 Date ""
@@
 	3750 1700 7750 1700
 $Comp
-L VCC #PWR0102
+L VCC #PWR101
 U 1 1 543F0201
 P 1050 950
-F 0 "#PWR0102" H 1050 1050 30  0001 C CNN
+F 0 "#PWR101" H 1050 1050 30  0001 C CNN
 F 1 "VCC" H 1050 1050 30  0000 C CNN
 F 2 "" H 1050 950 60  0000 C CNN
@@
 $EndComp
 $Comp
-L DGND #PWR0103
+L DGND #PWR102
 U 1 1 543F021F
 P 2500 3250
-F 0 "#PWR0103" H 2500 3250 40  0001 C CNN
+F 0 "#PWR102" H 2500 3250 40  0001 C CNN
 F 1 "DGND" H 2500 3180 40  0000 C CNN
 F 2 "" H 2500 3250 60  0000 C CNN
@@
 Text Notes 8050 4600 0    60   ~ 0
 Bi color leds : which button cap to get ?\n - Can't take the transparent red one or green led could be "ugly"\n - Transparent white could be ugly on its own...
-Text Notes 5650 5750 0    60   ~ 0
+Text Notes 5650 6450 0    60   ~ 0
 With single color leds, AS1115 can drive the loops state leds. This eliminate the needs of an additionnal MCP23017.\nThe button led resistances needs to be adjusted though (an additionnal resistance for each led ?)
 $Comp
@@
 Connection ~ 5050 4800
 Connection ~ 5050 5050
-Connection ~ 5050 5300
-Wire Wire Line
-	5050 3550 5050 5500
-Wire Wire Line
-	5050 5500 3750 5500
-Wire Wire Line
-	3750 5500 3750 2700
-Wire Wire Line
-	3750 2700 3450 2700
-Wire Bus Line
-	4050 2750 4050 5200
+Wire Bus Line
+	4050 2750 4050 5950
 $Comp
 L SW_TACT_LED SW12
@@
 	5550 5200 5650 5300
 Wire Bus Line
-	5550 3150 5550 5200
-Wire Bus Line
 	7750 3650 7400 3650
 NoConn ~ 3450 1500
@@
 Wire Bus Line
 	4150 3150 5550 3150
+$Comp
+L SW_TACT_LED SW20
+U 1 1 5473DCF9
+P 4750 5750
+F 0 "SW20" H 4550 5900 60  0000 C CNN
+F 1 "SW_TACT_LED" H 4720 5650 60  0001 C CNN
+F 2 "" H 4750 5750 60  0000 C CNN
+F 3 "" H 4750 5750 60  0000 C CNN
+	1    4750 5750
+	1    0    0    -1
+$EndComp
+$Comp
+L SW_TACT_LED SW21
+U 1 1 5473DD5D
+P 4750 6050
+F 0 "SW21" H 4550 6200 60  0000 C CNN
+F 1 "SW_TACT_LED" H 4720 5950 60  0001 C CNN
+F 2 "" H 4750 6050 60  0000 C CNN
+F 3 "" H 4750 6050 60  0000 C CNN
+	1    4750 6050
+	1    0    0    -1
+$EndComp
+Wire Wire Line
+	5050 5750 5050 6200
+Connection ~ 5050 6050
+Entry Wire Line
+	4050 5650 4150 5750
+Entry Wire Line
+	4050 5950 4150 6050
+Wire Wire Line
+	5050 5750 4950 5750
+Wire Wire Line
+	5050 6050 4950 6050
+Wire Wire Line
+	4450 5750 4150 5750
+Wire Wire Line
+	4450 6050 4150 6050
+Text Label 4450 5750 2    60   ~ 0
+SEGE
+Text Label 4450 6050 2    60   ~ 0
+SEGF
+Wire Wire Line
+	5050 3300 5050 5300
+Wire Wire Line
+	5050 3300 3450 3300
+Wire Wire Line
+	3450 3300 3450 2800
+Connection ~ 5050 3550
+Wire Wire Line
+	3450 2700 3750 2700
+Wire Wire Line
+	3750 2700 3750 6200
+Wire Wire Line
+	3750 6200 5050 6200
+Wire Bus Line
+	5550 3150 5550 5200
 $EndSCHEMATC
