File: mls800_front_panel.sch (KiCad schematic (older format))
At the start: 21 parts, among them SW12 SW_TACT_LED, SW13 SW_TACT_LED, SW14 SW_TACT_LED, SW15 SW_TACT_LED, SW16 SW_TACT_LED, SW17 SW_TACT_LED, SW18 SW_TACT_LED, SW19 SW_TACT_LED, SW20 SW_TACT_LED, SW21 SW_TACT_LED, U6 AS1115

Commit message: MLS800
* removed unnecessary filter on AVCC & AVCC1
* removed AREF connection
Parts:
- renumbered R27 to R19, R28 to R20, R29 to R21, R30 to R22, R31 to R23, R32 to R24, R33 to R25, R34 to R26, R35 to R27, SW18 to SW10, SW20 to SW10, SW19 to SW11, SW21 to SW11, SW12 to SW2, SW13 to SW3, SW14 to SW4, SW12 to SW4, SW15 to SW5, SW13 to SW5, SW16 to SW6, SW14 to SW6, SW17 to SW7, SW15 to SW7, SW18 to SW8, SW16 to SW8, SW19 to SW9, SW17 to SW9, U6 to U5
Changed lines of the file:
@@
 $Descr A4 11693 8268
 encoding utf-8
-Sheet 4 3
+Sheet 3 3
 Title ""
 Date ""
@@
 $EndComp
 $Comp
-L AS1115 U6
+L AS1115 U5
 U 1 1 543EEFD5
 P 2500 1900
-F 0 "U6" H 1950 3000 50  0000 C CNN
+F 0 "U5" H 1950 3000 50  0000 C CNN
 F 1 "AS1115" H 2950 800 50  0000 C CNN
 F 2 "MODULE" H 2000 800 50  0001 C CNN
@@
 	3750 1700 7750 1700
 $Comp
-L VCC #PWR101
+L VCC #PWR090
 U 1 1 543F0201
 P 1050 950
-F 0 "#PWR101" H 1050 1050 30  0001 C CNN
+F 0 "#PWR090" H 1050 1050 30  0001 C CNN
 F 1 "VCC" H 1050 1050 30  0000 C CNN
 F 2 "" H 1050 950 60  0000 C CNN
@@
 $EndComp
 $Comp
-L DGND #PWR102
+L DGND #PWR091
 U 1 1 543F021F
 P 2500 3250
-F 0 "#PWR102" H 2500 3250 40  0001 C CNN
+F 0 "#PWR091" H 2500 3250 40  0001 C CNN
 F 1 "DGND" H 2500 3180 40  0000 C CNN
 F 2 "" H 2500 3250 60  0000 C CNN
@@
 IRQ
 $Comp
-L R R27
+L R R19
 U 1 1 543F1E5E
 P 1300 1050
-F 0 "R27" V 1380 1050 40  0000 C CNN
+F 0 "R19" V 1380 1050 40  0000 C CNN
 F 1 "R" V 1307 1051 40  0000 C CNN
 F 2 "" V 1230 1050 30  0000 C CNN
@@
 With single color leds, AS1115 can drive the loops state leds. This eliminate the needs of an additionnal MCP23017.\nThe button led resistances needs to be adjusted though (an additionnal resistance for each led ?)
 $Comp
-L SW_TACT_LED SW12
+L SW_TACT_LED SW2
 U 1 1 54402E3F
 P 4750 3550
-F 0 "SW12" H 4550 3700 60  0000 C CNN
+F 0 "SW2" H 4550 3700 60  0000 C CNN
 F 1 "SW_TACT_LED" H 4720 3450 60  0001 C CNN
 F 2 "" H 4750 3550 60  0000 C CNN
@@
 $EndComp
 $Comp
-L SW_TACT_LED SW13
+L SW_TACT_LED SW3
 U 1 1 54402F2D
 P 4750 3800
-F 0 "SW13" H 4550 3950 60  0000 C CNN
+F 0 "SW3" H 4550 3950 60  0000 C CNN
 F 1 "SW_TACT_LED" H 4720 3700 60  0001 C CNN
 F 2 "" H 4750 3800 60  0000 C CNN
@@
 $EndComp
 $Comp
-L SW_TACT_LED SW14
+L SW_TACT_LED SW4
 U 1 1 54402F4E
 P 4750 4050
-F 0 "SW14" H 4550 4200 60  0000 C CNN
+F 0 "SW4" H 4550 4200 60  0000 C CNN
 F 1 "SW_TACT_LED" H 4720 3950 60  0001 C CNN
 F 2 "" H 4750 4050 60  0000 C CNN
@@
 $EndComp
 $Comp
-L SW_TACT_LED SW15
+L SW_TACT_LED SW5
 U 1 1 54402F70
 P 4750 4300
-F 0 "SW15" H 4550 4450 60  0000 C CNN
+F 0 "SW5" H 4550 4450 60  0000 C CNN
 F 1 "SW_TACT_LED" H 4720 4200 60  0001 C CNN
 F 2 "" H 4750 4300 60  0000 C CNN
@@
 $EndComp
 $Comp
-L SW_TACT_LED SW16
+L SW_TACT_LED SW6
 U 1 1 54402F97
 P 4750 4550
-F 0 "SW16" H 4550 4700 60  0000 C CNN
+F 0 "SW6" H 4550 4700 60  0000 C CNN
 F 1 "SW_TACT_LED" H 4720 4450 60  0001 C CNN
 F 2 "" H 4750 4550 60  0000 C CNN
@@
 $EndComp
 $Comp
-L SW_TACT_LED SW17
+L SW_TACT_LED SW7
 U 1 1 54403051
 P 4750 4800
-F 0 "SW17" H 4550 4950 60  0000 C CNN
+F 0 "SW7" H 4550 4950 60  0000 C CNN
 F 1 "SW_TACT_LED" H 4720 4700 60  0001 C CNN
 F 2 "" H 4750 4800 60  0000 C CNN
@@
 $EndComp
 $Comp
-L SW_TACT_LED SW18
+L SW_TACT_LED SW8
 U 1 1 54403086
 P 4750 5050
-F 0 "SW18" H 4550 5200 60  0000 C CNN
+F 0 "SW8" H 4550 5200 60  0000 C CNN
 F 1 "SW_TACT_LED" H 4720 4950 60  0001 C CNN
 F 2 "" H 4750 5050 60  0000 C CNN
@@
 $EndComp
 $Comp
-L SW_TACT_LED SW19
+L SW_TACT_LED SW9
 U 1 1 544030B0
 P 4750 5300
-F 0 "SW19" H 4550 5450 60  0000 C CNN
+F 0 "SW9" H 4550 5450 60  0000 C CNN
 F 1 "SW_TACT_LED" H 4720 5200 60  0001 C CNN
 F 2 "" H 4750 5300 60  0000 C CNN
@@
 	4050 2750 4050 5950
 $Comp
-L SW_TACT_LED SW12
+L SW_TACT_LED SW4
 U 2 1 54405D5F
 P 6850 3550
-F 0 "SW12" H 6650 3700 60  0000 C CNN
+F 0 "SW4" H 6650 3700 60  0000 C CNN
 F 1 "SW_TACT_LED" H 6820 3450 60  0001 C CNN
 F 2 "" H 6850 3550 60  0000 C CNN
@@
 $EndComp
 $Comp
-L SW_TACT_LED SW13
+L SW_TACT_LED SW5
 U 2 1 54405E2B
 P 6850 3800
-F 0 "SW13" H 6650 3950 60  0000 C CNN
+F 0 "SW5" H 6650 3950 60  0000 C CNN
 F 1 "SW_TACT_LED" H 6820 3700 60  0001 C CNN
 F 2 "" H 6850 3800 60  0000 C CNN
@@
 $EndComp
 $Comp
-L SW_TACT_LED SW14
+L SW_TACT_LED SW6
 U 2 1 54405E54
 P 6850 4050
-F 0 "SW14" H 6650 4200 60  0000 C CNN
+F 0 "SW6" H 6650 4200 60  0000 C CNN
 F 1 "SW_TACT_LED" H 6820 3950 60  0001 C CNN
 F 2 "" H 6850 4050 60  0000 C CNN
@@
 $EndComp
 $Comp
-L SW_TACT_LED SW15
+L SW_TACT_LED SW7
 U 2 1 54405E7E
 P 6850 4300
-F 0 "SW15" H 6650 4450 60  0000 C CNN
+F 0 "SW7" H 6650 4450 60  0000 C CNN
 F 1 "SW_TACT_LED" H 6820 4200 60  0001 C CNN
 F 2 "" H 6850 4300 60  0000 C CNN
@@
 $EndComp
 $Comp
-L SW_TACT_LED SW16
+L SW_TACT_LED SW8
 U 2 1 54405EA9
 P 6850 4550
-F 0 "SW16" H 6650 4700 60  0000 C CNN
+F 0 "SW8" H 6650 4700 60  0000 C CNN
 F 1 "SW_TACT_LED" H 6820 4450 60  0001 C CNN
 F 2 "" H 6850 4550 60  0000 C CNN
@@
 $EndComp
 $Comp
-L SW_TACT_LED SW17
+L SW_TACT_LED SW9
 U 2 1 54405ED5
 P 6850 4800
-F 0 "SW17" H 6650 4950 60  0000 C CNN
+F 0 "SW9" H 6650 4950 60  0000 C CNN
 F 1 "SW_TACT_LED" H 6820 4700 60  0001 C CNN
 F 2 "" H 6850 4800 60  0000 C CNN
@@
 $EndComp
 $Comp
-L SW_TACT_LED SW18
+L SW_TACT_LED SW10
 U 2 1 54405F27
 P 6850 5050
-F 0 "SW18" H 6650 5200 60  0000 C CNN
+F 0 "SW10" H 6650 5200 60  0000 C CNN
 F 1 "SW_TACT_LED" H 6820 4950 60  0001 C CNN
 F 2 "" H 6850 5050 60  0000 C CNN
@@
 $EndComp
 $Comp
-L SW_TACT_LED SW19
+L SW_TACT_LED SW11
 U 2 1 54405F59
 P 6850 5300
-F 0 "SW19" H 6650 5450 60  0000 C CNN
+F 0 "SW11" H 6650 5450 60  0000 C CNN
 F 1 "SW_TACT_LED" H 6820 5200 60  0001 C CNN
 F 2 "" H 6850 5300 60  0000 C CNN
@@
 SEGDP
 $Comp
-L R R28
+L R R20
 U 1 1 54406B24
 P 6200 3550
-F 0 "R28" V 6280 3550 40  0000 C CNN
+F 0 "R20" V 6280 3550 40  0000 C CNN
 F 1 "110R" V 6207 3551 40  0000 C CNN
 F 2 "" V 6130 3550 30  0000 C CNN
@@
 $EndComp
 $Comp
-L R R29
+L R R21
 U 1 1 54408199
 P 6200 3800
-F 0 "R29" V 6280 3800 40  0000 C CNN
+F 0 "R21" V 6280 3800 40  0000 C CNN
 F 1 "110R" V 6207 3801 40  0000 C CNN
 F 2 "" V 6130 3800 30  0000 C CNN
@@
 $EndComp
 $Comp
-L R R30
+L R R22
 U 1 1 544081CA
 P 6200 4050
-F 0 "R30" V 6280 4050 40  0000 C CNN
+F 0 "R22" V 6280 4050 40  0000 C CNN
 F 1 "110R" V 6207 4051 40  0000 C CNN
 F 2 "" V 6130 4050 30  0000 C CNN
@@
 $EndComp
 $Comp
-L R R31
+L R R23
 U 1 1 5440822C
 P 6200 4300
-F 0 "R31" V 6280 4300 40  0000 C CNN
+F 0 "R23" V 6280 4300 40  0000 C CNN
 F 1 "110R" V 6207 4301 40  0000 C CNN
 F 2 "" V 6130 4300 30  0000 C CNN
@@
 $EndComp
 $Comp
-L R R32
+L R R24
 U 1 1 5440826B
 P 6200 4550
-F 0 "R32" V 6280 4550 40  0000 C CNN
+F 0 "R24" V 6280 4550 40  0000 C CNN
 F 1 "110R" V 6207 4551 40  0000 C CNN
 F 2 "" V 6130 4550 30  0000 C CNN
@@
 $EndComp
 $Comp
-L R R33
+L R R25
 U 1 1 5440829F
 P 6200 4800
-F 0 "R33" V 6280 4800 40  0000 C CNN
+F 0 "R25" V 6280 4800 40  0000 C CNN
 F 1 "110R" V 6207 4801 40  0000 C CNN
 F 2 "" V 6130 4800 30  0000 C CNN
@@
 $EndComp
 $Comp
-L R R34
+L R R26
 U 1 1 544082E4
 P 6200 5050
-F 0 "R34" V 6280 5050 40  0000 C CNN
+F 0 "R26" V 6280 5050 40  0000 C CNN
 F 1 "110R" V 6207 5051 40  0000 C CNN
 F 2 "" V 6130 5050 30  0000 C CNN
@@
 $EndComp
 $Comp
-L R R35
+L R R27
 U 1 1 5440831E
 P 6200 5300
-F 0 "R35" V 6280 5300 40  0000 C CNN
+F 0 "R27" V 6280 5300 40  0000 C CNN
 F 1 "110R" V 6207 5301 40  0000 C CNN
 F 2 "" V 6130 5300 30  0000 C CNN
@@
 	4150 3150 5550 3150
 $Comp
-L SW_TACT_LED SW20
+L SW_TACT_LED SW10
 U 1 1 5473DCF9
 P 4750 5750
-F 0 "SW20" H 4550 5900 60  0000 C CNN
+F 0 "SW10" H 4550 5900 60  0000 C CNN
 F 1 "SW_TACT_LED" H 4720 5650 60  0001 C CNN
 F 2 "" H 4750 5750 60  0000 C CNN
@@
 $EndComp
 $Comp
-L SW_TACT_LED SW21
+L SW_TACT_LED SW11
 U 1 1 5473DD5D
 P 4750 6050
-F 0 "SW21" H 4550 6200 60  0000 C CNN
+F 0 "SW11" H 4550 6200 60  0000 C CNN
 F 1 "SW_TACT_LED" H 4720 5950 60  0001 C CNN
 F 2 "" H 4750 6050 60  0000 C CNN
